File: ai-files/candidates/Battery_Charger.kicad_sch (KiCad schematic)
At the start: 35 parts, among them J5 1S_PACK_3PIN, Q100 2N7002, Q101 2N7002, Q102 2N7002, Q103 CSD17579Q3A, SW100 WAKE_QON, SW101 BAT_DISCONNECT, U4 BQ25792RQMR

Commit message: Checkpoint isolated BQ25792/TPS25730D/TPS2116 candidates, Q100 metadata and tool wrappers
Co-Authored-By: Claude Sonnet 5.5 <noreply@anthropic.com>
Parts:
- C110: LCSC (none) -> C107093; LCSC Part (none) -> C107093; MPN (none) -> CC0603KRX7R9BB473; Manufacturer (none) -> YAGEO
- C113, C114: LCSC (none) -> C1711; LCSC Part (none) -> C1711; MPN (none) -> CL21B104KBCNNNC; Manufacturer (none) -> Samsung Electro-Mechanics
- Q101, Q102: LCSC Part (none) -> C65189; MPN (none) -> 2N7002,215; Manufacturer (none) -> Nexperia
- R102: LCSC C107696 -> C99782; MPN RC0603FR-07220RL -> RC0603FR-074K7L
- R108: LCSC (none) -> C123419; MPN (none) -> RC0603FR-07180KL; Manufacturer (none) -> YAGEO
- R109, R110, R111: LCSC (none) -> C14675; MPN (none) -> RC0603FR-07100KL; Manufacturer (none) -> YAGEO
- R112: LCSC (none) -> C105588; MPN (none) -> RC0603FR-07100RL; Manufacturer (none) -> YAGEO
Connections:
- net BAT_INT is gone; now on net SYS_RAW: C106.1, Q103.[1-3] (S), U4.[22-23] (BAT)
- net PROG is gone; now on net REGN: R102.1, U4.20 (PROG)
- net TS_SENSE is gone; now on net BAT_PACK: J5.2 (Pin_2), R100.2, R101.1, U4.16 (TS)
- net BAT_PACK: now also J5.1 (Pin_1), SW101.2 (B)
- net CHG_VIO_3V0: now also R103.2, U4.13 (~{CE})
- net REGN: no longer C102.1, C109.1, U4.5 (REGN)
- net VBUS_PD: no longer U4.8 (VAC2), U4.9 (VAC1)
- removed net CE_N: Q100.3 (D), R103.2, U4.13 (~{CE})
- net ILIM_HIZ: no longer names the net of Q101.3 (D), R108.2, R109.1, U4.17 (HIZ/ILIM)
- net PMID: no longer names the net of C101.1, C108.1, C112.1, C114.1, U4.29 (PMID)
- net QON_SW: no longer names the net of SW100.1, U4.12 (QON)
- net SDRV: no longer names the net of Q103.4 (G), U4.24 (SDRV)
- net SW1: no longer names the net of C103.2, L1.1, U4.28 (SW1)
- net SW2: no longer names the net of C110.2, L1.2, U4.26 (SW2)
- new net: C102.1, C109.1, U4.5 (REGN)
Other:
- note added: "L1 2.2uH/6A and input MLCCs are provisional: qualify 20V surge/DC-bias, audio+charge current, ripple, efficiency and thermal limits."
- note added: "R102 4.7k = 1S/750kHz; use 1A initial charge target. D+/D− stay raw for mux. SYS_RAW varies; qualify TPS2116 5.5V limit/transients."
- note added: "Set REG14.SFET_PRESENT=1 before SDRV ship control. MCU reset/REG_RST requires reconfiguration. Pack 10k NTC curve and QON timing pending."
- note added: "Startup: keep HIZ clamped through POR; clear EN_EXTILIM, program/read back IINDPM and 1S limits before enabling SYS. Verify reset/watchdog recovery."
- note removed: "1S Li-ion; PROG 4.7k = 750kHz. Charge target 1A is firmware-only; POR 2A must remain disabled."
- note removed: "50uF nominal BQ bank counts in PD bulk budget; keep shared nominal bank <=100uF."
- note removed: "DP/DM left ports require a source-selection mux; do not tie to codec. SYS_RAW is variable NVDC, not 5V."
- note removed: "Do not release CHG_SYS_ENABLE before source-specific IINDPM. Prove REG_RST/watchdog behavior in firmware."
- note removed: "ILIM_HIZ low keeps switching off; POR sample below1.08V caches100mA. EN_EXTILIM/watchdog policy unresolved."
- note removed: "L1 2.2uH/6A is provisional: total SYS + charge current and ripple need product-load/thermal review."
- note removed: "PMID follows high input path: 35V caps shown; verify effective capacitance, derating and surge."
- note removed: "Pack and 10k NTC profile pending. QON wake defaults to ~1s low (15ms if configured); verify button hold."
- note removed: "TPS2116 SYS max5.5V; 1S default4.27–4.55V at BAT4.2; SYSMIN 3.5–4.1V; qualify SYSOVP/transients."
- moved on the sheet: C100, C101, C102, C103, C104, C105, C106, C107, C108, C109, J5, L1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

Commit message: Redraw TPS25730D and BQ25792 candidates readable; record handoffs and 5-20 V PD scope decision
Co-Authored-By: Claude Sonnet 5.5 <noreply@anthropic.com>
Connections:
- net BAT_PACK: no longer J5.1 (Pin_1), J5.2 (Pin_2), R100.2, R101.1, SW101.2 (B), U4.16 (TS)
- net CHG_VIO_3V0: no longer R103.2, U4.13 (~{CE})
- net REGN: now also C102.1, C109.1, U4.5 (REGN); no longer R102.1, U4.20 (PROG)
- net SYS_RAW: no longer C106.1, Q103.[1-3] (S), U4.[22-23] (BAT)
- net VBUS_PD: now also U4.8 (VAC2), U4.9 (VAC1)
- net PMID: now reaches C101.1, C108.1, C112.1, C114.1, U4.29 (PMID)
- net ILIM_HIZ: now reaches Q101.3 (D), R108.2, R109.1, U4.17 (ILIM_HIZ)
- net BTST2: now reaches C110.1, U4.19 (BTST2)
- net SW2: now reaches C110.2, L1.2, U4.26 (SW2)
- net SW1: now reaches C103.2, L1.1, U4.28 (SW1)
- net BTST1: now reaches C103.1, U4.4 (BTST1)
- net CE_N: now reaches Q100.3 (D)
- net CE_N: now also R103.2, U4.13 (~{CE})
- net BATP_SENSE: no longer names the net of R112.2, U4.18 (BATP)
- net Q101_GATE: no longer names the net of Q101.1 (G), Q102.3 (D), R110.2
- new net BAT_INT: C106.1, Q103.[1-3] (S), U4.[22-23] (BAT)
- new net PACK_RAW: J5.1 (Pin_1), SW101.2 (B)
- new net PROG: R102.1, U4.20 (PROG)
- new net TS_SENSE: J5.2 (Pin_2), R100.2, R101.1, U4.16 (TS)
Other:
- note added: "Config and default-off gates"
- note added: "I2C pull-ups (10k to logic rail) and CHG_VIO_3V0 level are host-side; D+/D- stay raw for later source-selection mux."
- note added: "R102 4.7k = 1S/750kHz PROG. L1 2.2uH/6A and input MLCCs are provisional: qualify 20V surge/DC-bias, load current, ripple, efficiency and thermal limits."
- note added: "Set REG14.SFET_PRESENT=1 and read back before SDRV ship control; POR default 0 locks SDRV_CTRL. MCU reset/REG_RST requires reconfiguration."
- note added: "Startup: keep ILIM_HIZ clamped (Q101) through POR; clear EN_EXTILIM, program/read back IINDPM and 1S limits before enabling SYS. Verify reset/watchdog recovery."
- note added: "VBUS input: VAC1/VAC2 tied to VBUS (no ACFETs); ACDRV1/2 to GND"
- note removed: "L1 2.2uH/6A and input MLCCs are provisional: qualify 20V surge/DC-bias, audio+charge current, ripple, efficiency and thermal limits."
- note removed: "R102 4.7k = 1S/750kHz; use 1A initial charge target. D+/D− stay raw for mux. SYS_RAW varies; qualify TPS2116 5.5V limit/transients."
- note removed: "Set REG14.SFET_PRESENT=1 before SDRV ship control. MCU reset/REG_RST requires reconfiguration. Pack 10k NTC curve and QON timing pending."
- note removed: "Startup: keep HIZ clamped through POR; clear EN_EXTILIM, program/read back IINDPM and 1S limits before enabling SYS. Verify reset/watchdog recovery."
- moved on the sheet: C100, C101, C102, C103, C104, C105, C106, C107, C108, C109, J5, L1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

Commit message: Apply Opus-reviewed must-fix items to PD and charger candidates
Co-Authored-By: Claude Sonnet 5.5 <noreply@anthropic.com>
Parts:
- added C115: 0.1uF / 50V, DesktopSpeaker:PD_C_0402, symbol PD_C:PD_C
- C113, C114: footprint DesktopSpeaker:PD_C_0603 -> DesktopSpeaker:PD_C_0402; LCSC C1711 -> C77020; LCSC Part C1711 -> C77020; MPN CL21B104KBCNNNC -> GRM155R71H104KE14D; Manufacturer Samsung Electro-Mechanics -> Murata
- R103: value 10k -> 100k; LCSC C98220 -> C14675; MPN RC0603FR-0710KL -> RC0603FR-07100KL
Connections:
- net GND: now also C115.2
- net SYS_RAW: now also C115.1
- net CHG_DM_RAW: no longer names the net of U4.7 (D−)
- net CHG_DP_RAW: no longer names the net of U4.6 (D+)
- no-connect marks 1 -> 3
Other:
- note added: "I2C pull-ups (10k to logic rail) and CHG_VIO_3V0 level are host-side; D+/D- unconnected (no-connect); set AUTO_INDET_EN=0, HVDCP_EN=0."
- note removed: "I2C pull-ups (10k to logic rail) and CHG_VIO_3V0 level are host-side; D+/D- stay raw for later source-selection mux."
- moved on the sheet: C104, C105, C107
