File: DesktopSpeaker-kicad/MCU.kicad_sch (KiCad schematic)
At the start: 9 parts, among them J6 SWD, J7 SWD_TC2030, U3 STM32G071RBT6

Commit message: Apply low-risk passive cuts (11 parts) and normalise BOM; add layout rules and BOM audit reports
Co-Authored-By: Claude Sonnet 5.5 <noreply@anthropic.com>
Claude-Session: https://claude.ai/code/session_01N5RHheWSjDFDPbKVD5YVeJ
Parts:
- removed C163: 100nF, DesktopSpeaker:C_0402_1005Metric_Pad0.74x0.62mm_HandSolder, symbol PD_C:PD_C
- removed C164: 1uF, DesktopSpeaker:C_0402_1005Metric_Pad0.74x0.62mm_HandSolder, symbol PD_C:PD_C
Changed lines of the file:
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@@
 (wire (pts (xy 134.62 66.04) (xy 139.7 66.04)) (stroke (width 0) (type default)))
 (wire (pts (xy 139.7 66.04) (xy 144.78 66.04)) (stroke (width 0) (type default)))
-(wire (pts (xy 144.78 66.04) (xy 152.4 66.04)) (stroke (width 0) (type default)))
-(wire (pts (xy 152.4 66.04) (xy 162.56 66.04)) (stroke (width 0) (type default)))
 (hierarchical_label "3V_AO" (shape input) (at 45.72 66.04 0) (effects (font (size 1.0 1.0)) (justify left bottom)))
 (junction (at 113.03 66.04) (diameter 0) (color 0 0 0 0))
@@
 (junction (at 134.62 66.04) (diameter 0) (color 0 0 0 0))
 (junction (at 139.7 66.04) (diameter 0) (color 0 0 0 0))
-(junction (at 152.4 66.04) (diameter 0) (color 0 0 0 0))
-(symbol (lib_id "PD_C:PD_C") (at 152.4 69.85 0) (unit 1) (exclude_from_sim no) (in_bom yes) (on_board yes) (dnp no) (property "Reference" "C163" (at 153.67 68.58 0) (effects (font (size 1.27 1.27)) (justify left))) (property "Value" "100nF" (at 153.67 71.12 0) (effects (font (size 1.27 1.27)) (justify left))) (property "Footprint" "DesktopSpeaker:C_0402_1005Metric_Pad0.74x0.62mm_HandSolder" (at 152.4 69.85 0) (hide yes) (effects (font (size 1.27 1.27)))) (property "MPN" "GRM155R71H104KE14D" (at 152.4 69.85 0) (hide yes) (effects (font (size 1.27 1.27)))) (property "Manufacturer" "Murata" (at 152.4 69.85 0) (hide yes) (effects (font (size 1 1)))) (property "LCSC" "C77020" (at 152.4 69.85 0) (hide yes) (effects (font (size 1 1)))) (property "Datasheet" "${KIPRJMOD}/../ai-files/datasheets/Samsung_MLCC_LCSC_C1591_C1711.pdf" (at 152.4 69.85 0) (hide yes) (effects (font (size 1 1)))) (pin "1") (pin "2") (instances (project "DesktopSpeaker" (path "/feda53ed-537d-4f88-9436-c6075776255b/4ab2b160-efba-45d8-be2c-c7b2862cfacf" (reference "C163") (unit 1)))))
-(symbol (lib_id "power:GND") (at 152.4 73.66 0) (unit 1) (exclude_from_sim no) (in_bom no) (on_board no) (dnp no) (property "Reference" "#PWR910" (at 152.4 77.47 0) (effects (font (size 1.27 1.27)) (hide yes))) (property "Value" "GND" (at 152.4 78.74 0) (effects (font (size 1.27 1.27)) (hide yes))) (pin "1") (instances (project "DesktopSpeaker" (path "/feda53ed-537d-4f88-9436-c6075776255b/4ab2b160-efba-45d8-be2c-c7b2862cfacf" (reference "#PWR910") (unit 1)))))
-(symbol (lib_id "PD_C:PD_C") (at 162.56 69.85 0) (unit 1) (exclude_from_sim no) (in_bom yes) (on_board yes) (dnp no) (property "Reference" "C164" (at 163.83 68.58 0) (effects (font (size 1.27 1.27)) (justify left))) (property "Value" "1uF" (at 163.83 71.12 0) (effects (font (size 1.27 1.27)) (justify left))) (property "Footprint" "DesktopSpeaker:C_0402_1005Metric_Pad0.74x0.62mm_HandSolder" (at 162.56 69.85 0) (hide yes) (effects (font (size 1.27 1.27)))) (property "MPN" "CL05A105KO5NNNC" (at 162.56 69.85 0) (hide yes) (effects (font (size 1.27 1.27)))) (property "Manufacturer" "Samsung Electro-Mechanics" (at 162.56 69.85 0) (hide yes) (effects (font (size 1 1)))) (property "LCSC" "C29266" (at 162.56 69.85 0) (hide yes) (effects (font (size 1 1)))) (property "Datasheet" "" (at 162.56 69.85 0) (hide yes) (effects (font (size 1 1)))) (pin "1") (pin "2") (instances (project "DesktopSpeaker" (path "/feda53ed-537d-4f88-9436-c6075776255b/4ab2b160-efba-45d8-be2c-c7b2862cfacf" (reference "C164") (unit 1)))))
-(symbol (lib_id "power:GND") (at 162.56 73.66 0) (unit 1) (exclude_from_sim no) (in_bom no) (on_board no) (dnp no) (property "Reference" "#PWR911" (at 162.56 77.47 0) (effects (font (size 1.27 1.27)) (hide yes))) (property "Value" "GND" (at 162.56 78.74 0) (effects (font (size 1.27 1.27)) (hide yes))) (pin "1") (instances (project "DesktopSpeaker" (path "/feda53ed-537d-4f88-9436-c6075776255b/4ab2b160-efba-45d8-be2c-c7b2862cfacf" (reference "#PWR911") (unit 1)))))
 (wire (pts (xy 129.54 168.91) (xy 129.54 171.45)) (stroke (width 0) (type default)))
 (symbol (lib_id "power:GND") (at 129.54 171.45 0) (unit 1) (exclude_from_sim no) (in_bom no) (on_board no) (dnp no) (property "Reference" "#PWR912" (at 129.54 175.26 0) (effects (font (size 1.27 1.27)) (hide yes))) (property "Value" "GND" (at 129.54 176.53 0) (effects (font (size 1.27 1.27)) (hide yes))) (pin "1") (instances (project "DesktopSpeaker" (path "/feda53ed-537d-4f88-9436-c6075776255b/4ab2b160-efba-45d8-be2c-c7b2862cfacf" (reference "#PWR912") (unit 1)))))
