File: DesktopSpeaker-kicad/Battery_Charger.kicad_sch (KiCad schematic)
At the start: 37 parts, among them J5 1S_PACK_3PIN, Q100 2N7002, Q101 2N7002, Q102 2N7002, Q103 CSD17579Q3A, SW100 WAKE_QON, SW101 BAT_DISCONNECT, U4 BQ25792RQMR

Commit message: Repackage passives to 0402/0805 hand-solder footprints; update BOM and flags
Co-Authored-By: Claude Sonnet 5.5 <noreply@anthropic.com>
Claude-Session: https://claude.ai/code/session_01N5RHheWSjDFDPbKVD5YVeJ
Parts:
- C100, C101, C108: footprint DesktopSpeaker:PD_C_1210 -> DesktopSpeaker:C_0805_2012Metric_Pad1.18x1.45mm_HandSolder; LCSC Part C138687 -> (none); MPN CL32B106KBJNNNE -> GRM21BR61H106KE43L; Manufacturer Samsung Electro-Mechanics -> Murata
- C102, C109: footprint DesktopSpeaker:PD_C_0805 -> DesktopSpeaker:C_0805_2012Metric_Pad1.18x1.45mm_HandSolder; LCSC (none) -> C32635
- C103, C110: footprint DesktopSpeaker:PD_C_0603 -> DesktopSpeaker:C_0402_1005Metric_Pad0.74x0.62mm_HandSolder; LCSC C107093 -> (none); LCSC Part C107093 -> (none); MPN CC0603KRX7R9BB473 -> GRM155R71H473KA12D; Manufacturer YAGEO -> Murata
- C104, C105, C106, C107: footprint DesktopSpeaker:PD_C_0805 -> DesktopSpeaker:C_0805_2012Metric_Pad1.18x1.45mm_HandSolder; LCSC (none) -> C907991
- C111, C112: footprint DesktopSpeaker:PD_C_1210 -> DesktopSpeaker:C_0805_2012Metric_Pad1.18x1.45mm_HandSolder; LCSC C138687 -> (none); LCSC Part C138687 -> (none); MPN CL32B106KBJNNNE -> GRM21BR61H106KE43L; Manufacturer Samsung Electro-Mechanics -> Murata
- C113, C114, C115: footprint DesktopSpeaker:PD_C_0402 -> DesktopSpeaker:C_0402_1005Metric_Pad0.74x0.62mm_HandSolder
- R100: footprint DesktopSpeaker:PD_R_0603 -> DesktopSpeaker:R_0402_1005Metric_Pad0.72x0.64mm_HandSolder; LCSC C54531489 -> (none); MPN 1RC0603F5231 -> RC0402FR-075K23L; Manufacturer SAE -> Yageo
- R101: footprint DesktopSpeaker:PD_R_0603 -> DesktopSpeaker:R_0402_1005Metric_Pad0.72x0.64mm_HandSolder; LCSC C54531365 -> (none); MPN 1RC0603F3012 -> RC0402FR-0730K1L; Manufacturer SAE -> Yageo
- R102: footprint DesktopSpeaker:PD_R_0603 -> DesktopSpeaker:R_0402_1005Metric_Pad0.72x0.64mm_HandSolder; LCSC C99782 -> (none); MPN RC0603FR-074K7L -> RC0402FR-074K7L; Manufacturer YAGEO -> Yageo
- R103, R107, R109, R110, R111, R113: footprint DesktopSpeaker:PD_R_0603 -> DesktopSpeaker:R_0402_1005Metric_Pad0.72x0.64mm_HandSolder; LCSC C14675 -> C60491; MPN RC0603FR-07100KL -> RC0402FR-07100KL; Manufacturer YAGEO -> Yageo
- R106: footprint DesktopSpeaker:PD_R_0603 -> DesktopSpeaker:R_0402_1005Metric_Pad0.72x0.64mm_HandSolder; LCSC C98220 -> C60490; MPN RC0603FR-0710KL -> RC0402FR-0710KL; Manufacturer YAGEO -> Yageo
- R108: footprint DesktopSpeaker:PD_R_0603 -> DesktopSpeaker:R_0402_1005Metric_Pad0.72x0.64mm_HandSolder; LCSC C123419 -> (none); MPN RC0603FR-07180KL -> RC0402FR-07180KL; Manufacturer YAGEO -> Yageo
- R112: footprint DesktopSpeaker:PD_R_0603 -> DesktopSpeaker:R_0402_1005Metric_Pad0.72x0.64mm_HandSolder; LCSC C105588 -> (none); MPN RC0603FR-07100RL -> RC0402FR-07100RL; Manufacturer YAGEO -> Yageo

Commit message: Apply low-risk passive cuts (11 parts) and normalise BOM; add layout rules and BOM audit reports
Co-Authored-By: Claude Sonnet 5.5 <noreply@anthropic.com>
Claude-Session: https://claude.ai/code/session_01N5RHheWSjDFDPbKVD5YVeJ
Parts:
- removed C113, C114, C115: 0.1uF / 50V, DesktopSpeaker:C_0402_1005Metric_Pad0.74x0.62mm_HandSolder, symbol PD_C:PD_C

Commit message: Placement v9: EC11E volume encoder, 25 test points, silkscreen pass (closed sections, border, hole squares, labels), Orwellian logo on back, CAD refit
Co-Authored-By: Claude Sonnet 5.5 <noreply@anthropic.com>
Claude-Session: https://claude.ai/code/session_016fe4xPJbEE2SjGafuyNLjb
Parts:
- added TP11: REGN, DesktopSpeaker:TestPoint_Keystone_5015_Micro_Mini, symbol TestPoint:TestPoint
- added TP2: SYS_RAW, DesktopSpeaker:TestPoint_Keystone_5015_Micro_Mini, symbol TestPoint:TestPoint
Connections:
- net REGN: now also TP11.1
- net SYS_RAW: now also TP2.1
Changed lines of the file:
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@@
 (label "CHG_QON_SENSE" (at 381.0 187.96 0) (effects (font (size 1 1)) (justify right bottom)))
 (hierarchical_label "CHG_QON_SENSE" (shape output) (at 391.16 187.96 0) (effects (font (size 1.0 1.0)) (justify right bottom)))
+(symbol (lib_id "TestPoint:TestPoint") (at 393.7 121.92 0) (unit 1) (exclude_from_sim no) (in_bom no) (on_board yes) (dnp no) (property "Reference" "TP2" (at 395.73 117.35 0) (effects (font (size 1.27 1.27)) (justify left))) (property "Value" "SYS_RAW" (at 395.73 119.89 0) (effects (font (size 1.27 1.27)) (justify left))) (property "Footprint" "DesktopSpeaker:TestPoint_Keystone_5015_Micro_Mini" (at 393.7 121.92 0) (hide yes) (effects (font (size 1.27 1.27)))) (property "Datasheet" "" (at 393.7 121.92 0) (hide yes) (effects (font (size 1.27 1.27)))) (property "Description" "Debug test point (excluded from BOM; hand-fitted loop)" (at 393.7 121.92 0) (hide yes) (effects (font (size 1 1)))) (pin "1") (instances (project "DesktopSpeaker" (path "/feda53ed-537d-4f88-9436-c6075776255b/a7066d55-4393-49f1-9dcb-c2e9f1db9549" (reference "TP2") (unit 1)))))
+(wire (pts (xy 393.7 121.92) (xy 393.7 124.46)) (stroke (width 0) (type default)))
+(label "SYS_RAW" (at 393.7 124.46 0) (effects (font (size 1 1)) (justify left bottom)))
+(symbol (lib_id "TestPoint:TestPoint") (at 248.92 93.98 0) (unit 1) (exclude_from_sim no) (in_bom no) (on_board yes) (dnp no) (property "Reference" "TP11" (at 250.95 89.41 0) (effects (font (size 1.27 1.27)) (justify left))) (property "Value" "REGN" (at 250.95 91.95 0) (effects (font (size 1.27 1.27)) (justify left))) (property "Footprint" "DesktopSpeaker:TestPoint_Keystone_5015_Micro_Mini" (at 248.92 93.98 0) (hide yes) (effects (font (size 1.27 1.27)))) (property "Datasheet" "" (at 248.92 93.98 0) (hide yes) (effects (font (size 1.27 1.27)))) (property "Description" "Debug test point (excluded from BOM; hand-fitted loop)" (at 248.92 93.98 0) (hide yes) (effects (font (size 1 1)))) (pin "1") (instances (project "DesktopSpeaker" (path "/feda53ed-537d-4f88-9436-c6075776255b/a7066d55-4393-49f1-9dcb-c2e9f1db9549" (reference "TP11") (unit 1)))))
+(wire (pts (xy 248.92 93.98) (xy 248.92 96.52)) (stroke (width 0) (type default)))
+(label "REGN" (at 248.92 96.52 0) (effects (font (size 1 1)) (justify left bottom)))
 )
