File: DesktopSpeaker-kicad/Battery_Charger.kicad_sch (KiCad schematic)
At the start: 36 parts, among them J5 1S_PACK_3PIN, Q100 2N7002, Q101 2N7002, Q102 2N7002, Q103 CSD17579Q3A, SW100 WAKE_QON, SW101 BAT_DISCONNECT, U4 BQ25792RQMR

Commit message: Schematic: add C311-C316, TP26/27; placement v10 to v10d (reviewed), reports and generators
Co-Authored-By: Claude Sonnet 5.5 <noreply@anthropic.com>
Claude-Session: https://claude.ai/code/session_016fe4xPJbEE2SjGafuyNLjb
Parts:
- added C311, C312, C313: 100nF, DesktopSpeaker:C_0402_1005Metric_Pad0.74x0.62mm_HandSolder, symbol PD_C:PD_C
- added TP26, TP27: GND, DesktopSpeaker:TestPoint_Keystone_5010-5014_Multipurpose, symbol TestPoint:TestPoint
Connections:
- net GND: now also C311.2, C312.2, C313.2, TP26.1, TP27.1
- net PMID: now also C312.1
- net SYS_RAW: now also C311.1
- net VBUS_PD: now also C313.1
Changed lines of the file:
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@@
 (symbol (lib_id "PD_PWR_FLAG:PD_PWR_FLAG") (at 259.08 142.24 0) (unit 1) (exclude_from_sim no) (in_bom no) (on_board no) (dnp no) (property "Reference" "#FLG211" (at 259.08 135.89 0) (hide yes) (effects (font (size 1.27 1.27)))) (property "Value" "PWR_FLAG" (at 259.08 138.43 0) (hide yes) (effects (font (size 1.27 1.27)))) (property "Footprint" "" (at 259.08 142.24 0) (hide yes) (effects (font (size 1.27 1.27)))) (property "Datasheet" "" (at 259.08 142.24 0) (hide yes) (effects (font (size 1.27 1.27)))) (pin "1") (instances (project "DesktopSpeaker" (path "/feda53ed-537d-4f88-9436-c6075776255b/a7066d55-4393-49f1-9dcb-c2e9f1db9549" (reference "#FLG211") (unit 1)))))
 (junction (at 259.08 142.24) (diameter 0) (color 0 0 0 0))
+(symbol (lib_id "PD_C:PD_C") (at 327.66 133.35 0) (unit 1) (exclude_from_sim no) (in_bom yes) (on_board yes) (dnp no) (property "Reference" "C311" (at 332.74 132.08 0) (effects (font (size 1.27 1.27)) (justify left))) (property "Value" "100nF" (at 332.74 134.62 0) (effects (font (size 1.27 1.27)) (justify left))) (property "Footprint" "DesktopSpeaker:C_0402_1005Metric_Pad0.74x0.62mm_HandSolder" (at 327.66 133.35 0) (effects (font (size 1.0 1.0)) (hide yes))) (property "LCSC" "" (at 327.66 133.35 0) (hide yes) (effects (font (size 1 1)))) (property "Manufacturer" "Murata" (at 327.66 133.35 0) (effects (font (size 1.0 1.0)) (hide yes))) (property "MPN" "GRM155R71H104KE14D" (at 327.66 133.35 0) (effects (font (size 1.0 1.0)) (hide yes))) (property "LCSC Part" "" (at 327.66 133.35 0) (effects (font (size 1.0 1.0)) (hide yes))) (property "Datasheet" "${KIPRJMOD}/../ai-files/datasheets/Samsung_MLCC_LCSC_C1591_C1711.pdf" (at 327.66 133.35 0) (effects (font (size 1.0 1.0)) (hide yes))) (pin "1") (pin "2") (instances (project "DesktopSpeaker" (path "/feda53ed-537d-4f88-9436-c6075776255b/a7066d55-4393-49f1-9dcb-c2e9f1db9549" (reference "C311") (unit 1)))))
+(symbol (lib_id "power:GND") (at 327.66 137.16 0) (unit 1) (exclude_from_sim no) (in_bom no) (on_board no) (dnp no) (property "Reference" "#PWR2001" (at 332.74 135.89 0) (effects (font (size 1.27 1.27)) (justify left) (hide yes))) (property "Value" "GND" (at 327.66 142.24 0) (effects (font (size 1.27 1.27)))) (property "Footprint" "" (at 328.93 160.02 0) (effects (font (size 1.0 1.0)) (hide yes))) (pin "1") (instances (project "DesktopSpeaker" (path "/feda53ed-537d-4f88-9436-c6075776255b/a7066d55-4393-49f1-9dcb-c2e9f1db9549" (reference "#PWR2001") (unit 1)))))
+(junction (at 327.66 129.54) (diameter 0) (color 0 0 0 0))
+(symbol (lib_id "PD_C:PD_C") (at 327.66 87.63 0) (unit 1) (exclude_from_sim no) (in_bom yes) (on_board yes) (dnp no) (property "Reference" "C312" (at 332.74 86.36 0) (effects (font (size 1.27 1.27)) (justify left))) (property "Value" "100nF" (at 332.74 88.9 0) (effects (font (size 1.27 1.27)) (justify left))) (property "Footprint" "DesktopSpeaker:C_0402_1005Metric_Pad0.74x0.62mm_HandSolder" (at 327.66 87.63 0) (effects (font (size 1.0 1.0)) (hide yes))) (property "LCSC" "" (at 327.66 87.63 0) (hide yes) (effects (font (size 1 1)))) (property "Manufacturer" "Murata" (at 327.66 87.63 0) (effects (font (size 1.0 1.0)) (hide yes))) (property "MPN" "GRM155R71H104KE14D" (at 327.66 87.63 0) (effects (font (size 1.0 1.0)) (hide yes))) (property "LCSC Part" "" (at 327.66 87.63 0) (effects (font (size 1.0 1.0)) (hide yes))) (property "Datasheet" "${KIPRJMOD}/../ai-files/datasheets/Samsung_MLCC_LCSC_C1591_C1711.pdf" (at 327.66 87.63 0) (effects (font (size 1.0 1.0)) (hide yes))) (pin "1") (pin "2") (instances (project "DesktopSpeaker" (path "/feda53ed-537d-4f88-9436-c6075776255b/a7066d55-4393-49f1-9dcb-c2e9f1db9549" (reference "C312") (unit 1)))))
+(symbol (lib_id "power:GND") (at 327.66 91.44 0) (unit 1) (exclude_from_sim no) (in_bom no) (on_board no) (dnp no) (property "Reference" "#PWR2002" (at 332.74 90.17 0) (effects (font (size 1.27 1.27)) (justify left) (hide yes))) (property "Value" "GND" (at 327.66 96.52 0) (effects (font (size 1.27 1.27)))) (property "Footprint" "" (at 328.93 114.3 0) (effects (font (size 1.0 1.0)) (hide yes))) (pin "1") (instances (project "DesktopSpeaker" (path "/feda53ed-537d-4f88-9436-c6075776255b/a7066d55-4393-49f1-9dcb-c2e9f1db9549" (reference "#PWR2002") (unit 1)))))
+(wire (pts (xy 304.8 83.82) (xy 327.66 83.82)) (stroke (width 0) (type default)))
+(junction (at 304.8 83.82) (diameter 0) (color 0 0 0 0))
+(symbol (lib_id "PD_C:PD_C") (at 187.96 105.41 0) (unit 1) (exclude_from_sim no) (in_bom yes) (on_board yes) (dnp no) (property "Reference" "C313" (at 193.04 104.14 0) (effects (font (size 1.27 1.27)) (justify left))) (property "Value" "100nF" (at 193.04 106.68 0) (effects (font (size 1.27 1.27)) (justify left))) (property "Footprint" "DesktopSpeaker:C_0402_1005Metric_Pad0.74x0.62mm_HandSolder" (at 187.96 105.41 0) (effects (font (size 1.0 1.0)) (hide yes))) (property "LCSC" "" (at 187.96 105.41 0) (hide yes) (effects (font (size 1 1)))) (property "Manufacturer" "Murata" (at 187.96 105.41 0) (effects (font (size 1.0 1.0)) (hide yes))) (property "MPN" "GRM155R71H104KE14D" (at 187.96 105.41 0) (effects (font (size 1.0 1.0)) (hide yes))) (property "LCSC Part" "" (at 187.96 105.41 0) (effects (font (size 1.0 1.0)) (hide yes))) (property "Datasheet" "${KIPRJMOD}/../ai-files/datasheets/Samsung_MLCC_LCSC_C1591_C1711.pdf" (at 187.96 105.41 0) (effects (font (size 1.0 1.0)) (hide yes))) (pin "1") (pin "2") (instances (project "DesktopSpeaker" (path "/feda53ed-537d-4f88-9436-c6075776255b/a7066d55-4393-49f1-9dcb-c2e9f1db9549" (reference "C313") (unit 1)))))
+(symbol (lib_id "power:GND") (at 187.96 109.22 0) (unit 1) (exclude_from_sim no) (in_bom no) (on_board no) (dnp no) (property "Reference" "#PWR2003" (at 193.04 107.95 0) (effects (font (size 1.27 1.27)) (justify left) (hide yes))) (property "Value" "GND" (at 187.96 114.3 0) (effects (font (size 1.27 1.27)))) (property "Footprint" "" (at 189.23 132.08 0) (effects (font (size 1.0 1.0)) (hide yes))) (pin "1") (instances (project "DesktopSpeaker" (path "/feda53ed-537d-4f88-9436-c6075776255b/a7066d55-4393-49f1-9dcb-c2e9f1db9549" (reference "#PWR2003") (unit 1)))))
+(junction (at 187.96 101.6) (diameter 0) (color 0 0 0 0))
+(symbol (lib_id "TestPoint:TestPoint") (at 299.72 50.8 0) (unit 1) (exclude_from_sim no) (in_bom no) (on_board yes) (dnp no) (property "Reference" "TP26" (at 302.57 46.23 0) (effects (font (size 1.27 1.27)) (justify left))) (property "Value" "GND" (at 302.57 48.77 0) (effects (font (size 1.27 1.27)) (justify left))) (property "Footprint" "DesktopSpeaker:TestPoint_Keystone_5010-5014_Multipurpose" (at 299.72 50.8 0) (hide yes) (effects (font (size 1.27 1.27)))) (property "Datasheet" "" (at 299.72 50.8 0) (hide yes) (effects (font (size 1.27 1.27)))) (property "Description" "Debug test point (excluded from BOM; hand-fitted loop)" (at 299.72 50.8 0) (hide yes) (effects (font (size 1 1)))) (pin "1") (instances (project "DesktopSpeaker" (path "/feda53ed-537d-4f88-9436-c6075776255b/a7066d55-4393-49f1-9dcb-c2e9f1db9549" (reference "TP26") (unit 1)))))
+(symbol (lib_id "power:GND") (at 299.72 53.34 0) (unit 1) (exclude_from_sim no) (in_bom no) (on_board no) (dnp no) (property "Reference" "#PWR2004" (at 305.62 52.07 0) (effects (font (size 1.27 1.27)) (justify left) (hide yes))) (property "Value" "GND" (at 299.72 58.42 0) (effects (font (size 1.27 1.27)))) (property "Footprint" "" (at 301.81 76.2 0) (effects (font (size 1.0 1.0)) (hide yes))) (pin "1") (instances (project "DesktopSpeaker" (path "/feda53ed-537d-4f88-9436-c6075776255b/a7066d55-4393-49f1-9dcb-c2e9f1db9549" (reference "#PWR2004") (unit 1)))))
+(wire (pts (xy 299.72 50.8) (xy 299.72 53.34)) (stroke (width 0) (type default)))
+(symbol (lib_id "TestPoint:TestPoint") (at 320.04 50.8 0) (unit 1) (exclude_from_sim no) (in_bom no) (on_board yes) (dnp no) (property "Reference" "TP27" (at 322.07 46.23 0) (effects (font (size 1.27 1.27)) (justify left))) (property "Value" "GND" (at 322.07 48.77 0) (effects (font (size 1.27 1.27)) (justify left))) (property "Footprint" "DesktopSpeaker:TestPoint_Keystone_5010-5014_Multipurpose" (at 320.04 50.8 0) (hide yes) (effects (font (size 1.27 1.27)))) (property "Datasheet" "" (at 320.04 50.8 0) (hide yes) (effects (font (size 1.27 1.27)))) (property "Description" "Debug test point (excluded from BOM; hand-fitted loop)" (at 320.04 50.8 0) (hide yes) (effects (font (size 1 1)))) (pin "1") (instances (project "DesktopSpeaker" (path "/feda53ed-537d-4f88-9436-c6075776255b/a7066d55-4393-49f1-9dcb-c2e9f1db9549" (reference "TP27") (unit 1)))))
+(symbol (lib_id "power:GND") (at 320.04 53.34 0) (unit 1) (exclude_from_sim no) (in_bom no) (on_board no) (dnp no) (property "Reference" "#PWR2005" (at 325.12 52.07 0) (effects (font (size 1.27 1.27)) (justify left) (hide yes))) (property "Value" "GND" (at 320.04 58.42 0) (effects (font (size 1.27 1.27)))) (property "Footprint" "" (at 321.31 76.2 0) (effects (font (size 1.0 1.0)) (hide yes))) (pin "1") (instances (project "DesktopSpeaker" (path "/feda53ed-537d-4f88-9436-c6075776255b/a7066d55-4393-49f1-9dcb-c2e9f1db9549" (reference "#PWR2005") (unit 1)))))
+(wire (pts (xy 320.04 50.8) (xy 320.04 53.34)) (stroke (width 0) (type default)))
 (sheet_instances (path "/" (page "1")))
 (embedded_fonts no)(wire (pts (xy 284.48 167.64) (xy 391.16 167.64)) (stroke (width 0) (type default)))

Commit message: Y200 24.576 MHz crystal with 15 pF load caps, C275 3D model, schematic/PCB sourcing fields synced to BOM
Co-Authored-By: Claude Sonnet 5.5 <noreply@anthropic.com>
Claude-Session: https://claude.ai/code/session_016fe4xPJbEE2SjGafuyNLjb
Parts:
- C100, C101, C108, C111, C112: LCSC (none) -> C440198; LCSC Part (none) -> C440198
- C103, C110: LCSC (none) -> C117757; LCSC Part (none) -> C117757; MPN GRM155R71H473KA12D -> GRM155R71H473KE14D
- C311, C312, C313: LCSC (none) -> C77020; LCSC Part (none) -> C77020
- Q100: LCSC (none) -> C65189; MPN (none) -> 2N7002,215; Manufacturer (none) -> Nexperia
- R100: LCSC (none) -> C25907; MPN RC0402FR-075K23L -> 0402WGF5231TCE; Manufacturer Yageo -> UNI-ROYAL
- R101: LCSC (none) -> C226982; MPN RC0402FR-0730K1L -> AC0402FR-0730K1L
- R102: LCSC (none) -> C105871
- R108: LCSC (none) -> C138046
- R112: LCSC (none) -> C106232
