File: DesktopSpeaker-kicad/Battery_Charger.kicad_sch (KiCad schematic)
At the start: 41 parts, among them J5 1S_PACK_3PIN, Q100 2N7002, Q101 2N7002, Q102 2N7002, Q103 CSD17579Q3A, SW100 WAKE_QON, SW101 BAT_DISCONNECT, U4 BQ25792RQMR

Commit message: Part substitutions from the sourcing pass: SW102 -> Alps EC11E18244AU (C202365, in stock), SW101 -> CW GRB112B802BR1 (Digi-Key, 20 A/14 VDC); sourcing report and Alps EC11E catalog
Co-Authored-By: Claude Fable 5.1 <noreply@anthropic.com>
Claude-Session: https://claude.ai/code/session_016fe4xPJbEE2SjGafuyNLjb
Parts:
- SW101: LCSC C5884429 -> (none); MPN KCD1-201-R -> GRB112B802BR1; Manufacturer SHOU HAN -> CW Industries
Changed lines of the file:
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@@
 (symbol (lib_id "PD_C:PD_C") (at 304.8 135.89 0) (unit 1) (exclude_from_sim no) (in_bom yes) (on_board yes) (dnp no) (property "Reference" "C106" (at 309.88 134.62 0) (effects (font (size 1.27 1.27)) (justify left))) (property "Value" "22uF / 10V" (at 309.88 137.16 0) (effects (font (size 1.27 1.27)) (justify left))) (property "Footprint" "DesktopSpeaker:C_0805_2012Metric_Pad1.18x1.45mm_HandSolder" (at 304.8 135.89 0) (effects (font (size 1.0 1.0)) (hide yes))) (property "LCSC" "C907991" (at 304.8 135.89 0) (hide yes) (effects (font (size 1 1)))) (property "Manufacturer" "Murata" (at 304.8 135.89 0) (effects (font (size 1.0 1.0)) (hide yes))) (property "MPN" "GRM21BZ71A226ME15L" (at 304.8 135.89 0) (effects (font (size 1.0 1.0)) (hide yes))) (property "LCSC Part" "C907991" (at 304.8 135.89 0) (effects (font (size 1.0 1.0)) (hide yes))) (property "Datasheet" "../ai-files/datasheets/Murata_GRM21BZ71A226ME15L_LCSC.pdf" (at 304.8 135.89 0) (effects (font (size 1.0 1.0)) (hide yes))) (pin "1") (pin "2") (instances (project "DesktopSpeaker" (path "/feda53ed-537d-4f88-9436-c6075776255b/a7066d55-4393-49f1-9dcb-c2e9f1db9549" (reference "C106") (unit 1)))))
 (symbol (lib_id "Connector_Generic:Conn_01x03") (at 345.44 154.94 0) (unit 1) (exclude_from_sim no) (in_bom yes) (on_board yes) (dnp no) (property "Reference" "J5" (at 350.52 153.67 0) (effects (font (size 1.27 1.27)) (justify left))) (property "Value" "1S_PACK_3PIN" (at 350.52 156.21 0) (effects (font (size 1.27 1.27)) (justify left))) (property "Footprint" "DesktopSpeaker:Molex_Micro-Fit_3.0_43650-0300_1x03_P3.00mm_Horizontal" (at 345.44 154.94 0) (effects (font (size 1.0 1.0)) (hide yes))) (property "Manufacturer" "Molex" (at 345.44 154.94 0) (effects (font (size 1.0 1.0)) (hide yes))) (property "MPN" "43650-0300" (at 345.44 154.94 0) (effects (font (size 1.0 1.0)) (hide yes))) (property "LCSC" "C503478" (at 345.44 154.94 0) (effects (font (size 1.0 1.0)) (hide yes))) (pin "1") (pin "2") (pin "3") (instances (project "DesktopSpeaker" (path "/feda53ed-537d-4f88-9436-c6075776255b/a7066d55-4393-49f1-9dcb-c2e9f1db9549" (reference "J5") (unit 1)))))
-(symbol (lib_id "Switch:SW_SPST") (at 307.34 152.4 0) (unit 1) (exclude_from_sim no) (in_bom yes) (on_board yes) (dnp no) (property "Reference" "SW101" (at 307.34 156.21 0) (effects (font (size 1.27 1.27)))) (property "Value" "BAT_DISCONNECT" (at 307.34 158.75 0) (effects (font (size 1.27 1.27)))) (property "Footprint" "DesktopSpeaker:SHOUHAN_KCD1-201-R_Rocker_D20_Panel" (at 307.34 152.4 0) (effects (font (size 1.0 1.0)) (hide yes))) (property "Manufacturer" "SHOU HAN" (at 307.34 152.4 0) (effects (font (size 1.0 1.0)) (hide yes))) (property "MPN" "KCD1-201-R" (at 307.34 152.4 0) (effects (font (size 1.0 1.0)) (hide yes))) (property "LCSC" "C5884429" (at 307.34 152.4 0) (effects (font (size 1.0 1.0)) (hide yes))) (pin "1") (pin "2") (instances (project "DesktopSpeaker" (path "/feda53ed-537d-4f88-9436-c6075776255b/a7066d55-4393-49f1-9dcb-c2e9f1db9549" (reference "SW101") (unit 1)))))
+(symbol (lib_id "Switch:SW_SPST") (at 307.34 152.4 0) (unit 1) (exclude_from_sim no) (in_bom yes) (on_board yes) (dnp no) (property "Reference" "SW101" (at 307.34 156.21 0) (effects (font (size 1.27 1.27)))) (property "Value" "BAT_DISCONNECT" (at 307.34 158.75 0) (effects (font (size 1.27 1.27)))) (property "Footprint" "DesktopSpeaker:SHOUHAN_KCD1-201-R_Rocker_D20_Panel" (at 307.34 152.4 0) (effects (font (size 1.0 1.0)) (hide yes))) (property "Manufacturer" "CW Industries" (at 307.34 152.4 0) (effects (font (size 1.0 1.0)) (hide yes))) (property "MPN" "GRB112B802BR1" (at 307.34 152.4 0) (effects (font (size 1.0 1.0)) (hide yes))) (property "LCSC" "" (at 307.34 152.4 0) (effects (font (size 1.0 1.0)) (hide yes))) (pin "1") (pin "2") (instances (project "DesktopSpeaker" (path "/feda53ed-537d-4f88-9436-c6075776255b/a7066d55-4393-49f1-9dcb-c2e9f1db9549" (reference "SW101") (unit 1)))))
 (symbol (lib_id "CSD17579Q3A:CSD17579Q3A") (at 271.78 137.16 0) (mirror x) (unit 1) (exclude_from_sim no) (in_bom yes) (on_board yes) (dnp no) (property "Reference" "Q103" (at 280.67 134.62 0) (effects (font (size 1.27 1.27)) (justify left))) (property "Value" "CSD17579Q3A" (at 280.67 137.16 0) (effects (font (size 1.27 1.27)) (justify left))) (property "Footprint" "DesktopSpeaker:CSD17579Q3A_DNH0008A" (at 271.78 137.16 0) (effects (font (size 1.0 1.0)) (hide yes))) (property "MPN" "CSD17579Q3A" (at 271.78 137.16 0) (effects (font (size 1.0 1.0)) (hide yes))) (property "LCSC Part" "C97376" (at 271.78 137.16 0) (effects (font (size 1.0 1.0)) (hide yes))) (property "Manufacturer" "Texas Instruments" (at 271.78 137.16 0) (effects (font (size 1.0 1.0)) (hide yes))) (property "Datasheet" "https://www.ti.com/lit/ds/symlink/csd17579q3a.pdf" (at 271.78 137.16 0) (effects (font (size 1.0 1.0)) (hide yes))) (pin "4") (pin "[1-3]") (pin "[5-9]") (instances (project "DesktopSpeaker" (path "/feda53ed-537d-4f88-9436-c6075776255b/a7066d55-4393-49f1-9dcb-c2e9f1db9549" (reference "Q103") (unit 1)))))
 (symbol (lib_id "PD_R:PD_R") (at 265.43 142.24 270) (unit 1) (exclude_from_sim no) (in_bom yes) (on_board yes) (dnp no) (property "Reference" "R112" (at 265.43 146.05 270) (effects (font (size 1.27 1.27)))) (property "Value" "100R" (at 265.43 148.59 270) (effects (font (size 1.27 1.27)))) (property "Footprint" "DesktopSpeaker:R_0402_1005Metric_Pad0.72x0.64mm_HandSolder" (at 265.43 142.24 0) (effects (font (size 1.0 1.0)) (hide yes))) (pin "1") (pin "2") (instances (project "DesktopSpeaker" (path "/feda53ed-537d-4f88-9436-c6075776255b/a7066d55-4393-49f1-9dcb-c2e9f1db9549" (reference "R112") (unit 1)))) (property "MPN" "RC0402FR-07100RL" (at 265.43 142.24 0) (effects (font (size 1 1)) (hide yes))) (property "Manufacturer" "Yageo" (at 265.43 142.24 0) (effects (font (size 1 1)) (hide yes))) (property "LCSC" "C106232" (at 265.43 142.24 0) (effects (font (size 1 1)) (hide yes))) (property "Datasheet" "${KIPRJMOD}/../ai-files/datasheets/Yageo_RC0603FR_series.pdf" (at 265.43 142.24 0) (effects (font (size 1 1)) (hide yes))))
