File: DesktopSpeaker-kicad/USB_PD.kicad_sch (KiCad schematic)
At the start: 23 parts, among them J4 I2C service, U11 TPS25730DREFR, U19 TPS7B8450QWDRBRQ1

Commit message: Apply low-risk passive cuts (11 parts) and normalise BOM; add layout rules and BOM audit reports
Co-Authored-By: Claude Sonnet 5.5 <noreply@anthropic.com>
Claude-Session: https://claude.ai/code/session_01N5RHheWSjDFDPbKVD5YVeJ
Parts:
- removed C185: 10uF X7R 10V CVIN_3V3, DesktopSpeaker:C_0805_2012Metric_Pad1.18x1.45mm_HandSolder, symbol PD_C:PD_C
Changed lines of the file:
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@@
 (symbol (lib_id "PD_C:PD_C") (at 170.18 54.61 0) (unit 1) (exclude_from_sim no) (in_bom yes) (on_board yes) (dnp no) (property "Reference" "C6" (at 173.99 53.34 0) (effects (font (size 1.27 1.27)) (justify left))) (property "Value" "22uF X7R 10V" (at 173.99 55.88 0) (effects (font (size 1.27 1.27)) (justify left))) (property "Footprint" "DesktopSpeaker:C_0805_2012Metric_Pad1.18x1.45mm_HandSolder" (at 170.18 54.61 0) (effects (font (size 1.27 1.27)) (hide yes))) (property "Datasheet" "" (at 170.18 54.61 0) (effects (font (size 1.27 1.27)) (hide yes))) (pin "1") (pin "2") (instances (project "DesktopSpeaker" (path "/feda53ed-537d-4f88-9436-c6075776255b/f38b7023-3d53-43ea-b3db-e2c826d87b35" (reference "C6") (unit 1)))) (property "Manufacturer" "Murata" (at 170.18 54.61 0) (effects (font (size 1.27 1.27)) (hide yes))) (property "MPN" "GRM21BZ71A226ME15L" (at 170.18 54.61 0) (effects (font (size 1.27 1.27)) (hide yes))) (property "LCSC Part" "C907991" (at 170.18 54.61 0) (effects (font (size 1.27 1.27)) (hide yes))) (property "LCSC" "C907991" (at 170.18 54.61 0) (effects (font (size 1.27 1.27)) (hide yes))))
 (symbol (lib_id "PD_C:PD_C") (at 195.58 54.61 0) (unit 1) (exclude_from_sim no) (in_bom yes) (on_board yes) (dnp no) (property "Reference" "C181" (at 199.39 53.34 0) (effects (font (size 1.27 1.27)) (justify left))) (property "Value" "10uF X7R 10V" (at 199.39 55.88 0) (effects (font (size 1.27 1.27)) (justify left))) (property "Footprint" "DesktopSpeaker:C_0805_2012Metric_Pad1.18x1.45mm_HandSolder" (at 195.58 54.61 0) (effects (font (size 1.27 1.27)) (hide yes))) (property "Datasheet" "" (at 195.58 54.61 0) (effects (font (size 1.27 1.27)) (hide yes))) (pin "1") (pin "2") (instances (project "DesktopSpeaker" (path "/feda53ed-537d-4f88-9436-c6075776255b/f38b7023-3d53-43ea-b3db-e2c826d87b35" (reference "C181") (unit 1)))) (property "Manufacturer" "Samsung Electro-Mechanics" (at 195.58 54.61 0) (effects (font (size 1.27 1.27)) (hide yes))) (property "MPN" "CL21B106KPQNNNE" (at 195.58 54.61 0) (effects (font (size 1.27 1.27)) (hide yes))) (property "LCSC Part" "C32635" (at 195.58 54.61 0) (effects (font (size 1.27 1.27)) (hide yes))) (property "LCSC" "C32635" (at 195.58 54.61 0) (effects (font (size 1.27 1.27)) (hide yes))) (property "Datasheet" "${KIPRJMOD}/../ai-files/datasheets/Samsung_CL21B106KPQNNNE.pdf" (at 195.58 54.61 0) (effects (font (size 1.27 1.27)) (hide yes))))
-(symbol (lib_id "PD_C:PD_C") (at 220.98 54.61 0) (unit 1) (exclude_from_sim no) (in_bom yes) (on_board yes) (dnp no) (property "Reference" "C185" (at 224.79 53.34 0) (effects (font (size 1.27 1.27)) (justify left))) (property "Value" "10uF X7R 10V CVIN_3V3" (at 224.79 55.88 0) (effects (font (size 1.27 1.27)) (justify left))) (property "Footprint" "DesktopSpeaker:C_0805_2012Metric_Pad1.18x1.45mm_HandSolder" (at 220.98 54.61 0) (effects (font (size 1.27 1.27)) (hide yes))) (property "Datasheet" "" (at 220.98 54.61 0) (effects (font (size 1.27 1.27)) (hide yes))) (pin "1") (pin "2") (instances (project "DesktopSpeaker" (path "/feda53ed-537d-4f88-9436-c6075776255b/f38b7023-3d53-43ea-b3db-e2c826d87b35" (reference "C185") (unit 1)))) (property "Manufacturer" "Samsung Electro-Mechanics" (at 220.98 54.61 0) (effects (font (size 1.27 1.27)) (hide yes))) (property "MPN" "CL21B106KPQNNNE" (at 220.98 54.61 0) (effects (font (size 1.27 1.27)) (hide yes))) (property "LCSC Part" "C32635" (at 220.98 54.61 0) (effects (font (size 1.27 1.27)) (hide yes))) (property "LCSC" "C32635" (at 220.98 54.61 0) (effects (font (size 1.27 1.27)) (hide yes))) (property "Datasheet" "${KIPRJMOD}/../ai-files/datasheets/Samsung_CL21B106KPQNNNE.pdf" (at 220.98 54.61 0) (effects (font (size 1.27 1.27)) (hide yes))))
 (symbol (lib_id "PD_C:PD_C") (at 50.8 110.49 0) (unit 1) (exclude_from_sim no) (in_bom yes) (on_board yes) (dnp no) (property "Reference" "C182" (at 54.61 109.22 0) (effects (font (size 1.27 1.27)) (justify left))) (property "Value" "330pF C0G CC1 filter" (at 54.61 111.76 0) (effects (font (size 1.27 1.27)) (justify left))) (property "Footprint" "DesktopSpeaker:C_0402_1005Metric_Pad0.74x0.62mm_HandSolder" (at 50.8 110.49 0) (effects (font (size 1.27 1.27)) (hide yes))) (property "LCSC" "" (at 50.8 110.49 0) (hide yes) (effects (font (size 1 1)))) (property "Datasheet" "" (at 50.8 110.49 0) (effects (font (size 1.27 1.27)) (hide yes))) (property "Manufacturer" "Murata" (at 50.8 110.49 0) (effects (font (size 1.27 1.27)) (hide yes))) (property "MPN" "GRM1555C1H331JA01D" (at 50.8 110.49 0) (effects (font (size 1.27 1.27)) (hide yes))) (property "LCSC Part" "" (at 50.8 110.49 0) (effects (font (size 1.27 1.27)) (hide yes))) (pin "1") (pin "2") (instances (project "DesktopSpeaker" (path "/feda53ed-537d-4f88-9436-c6075776255b/f38b7023-3d53-43ea-b3db-e2c826d87b35" (reference "C182") (unit 1)))))
 (symbol (lib_id "PD_C:PD_C") (at 50.8 123.19 0) (unit 1) (exclude_from_sim no) (in_bom yes) (on_board yes) (dnp no) (property "Reference" "C183" (at 54.61 121.92 0) (effects (font (size 1.27 1.27)) (justify left))) (property "Value" "330pF C0G CC2 filter" (at 54.61 124.46 0) (effects (font (size 1.27 1.27)) (justify left))) (property "Footprint" "DesktopSpeaker:C_0402_1005Metric_Pad0.74x0.62mm_HandSolder" (at 50.8 123.19 0) (effects (font (size 1.27 1.27)) (hide yes))) (property "LCSC" "" (at 50.8 123.19 0) (hide yes) (effects (font (size 1 1)))) (property "Datasheet" "" (at 50.8 123.19 0) (effects (font (size 1.27 1.27)) (hide yes))) (property "Manufacturer" "Murata" (at 50.8 123.19 0) (effects (font (size 1.27 1.27)) (hide yes))) (property "MPN" "GRM1555C1H331JA01D" (at 50.8 123.19 0) (effects (font (size 1.27 1.27)) (hide yes))) (property "LCSC Part" "" (at 50.8 123.19 0) (effects (font (size 1.27 1.27)) (hide yes))) (pin "1") (pin "2") (instances (project "DesktopSpeaker" (path "/feda53ed-537d-4f88-9436-c6075776255b/f38b7023-3d53-43ea-b3db-e2c826d87b35" (reference "C183") (unit 1)))))
@@
 (wire (pts (xy 220.98 50.8) (xy 220.98 48.26)) (stroke (width 0) (type default)))
 (label "VIN_LOW" (at 220.98 48.26 0) (effects (font (size 1 1)) (justify left bottom)))
-(symbol (lib_id "power:GND") (at 220.98 58.42 0) (unit 1) (exclude_from_sim no) (in_bom no) (on_board no) (dnp no) (property "Reference" "#PWR09" (at 220.98 54.42 0) (effects (font (size 1.27 1.27)) (hide yes))) (property "Value" "GND" (at 220.98 62.23 0) (effects (font (size 1.27 1.27)))) (property "Footprint" "" (at 220.98 58.42 0) (effects (font (size 1.27 1.27)) (hide yes))) (property "Datasheet" "" (at 220.98 58.42 0) (effects (font (size 1.27 1.27)) (hide yes))) (pin "1") (instances (project "DesktopSpeaker" (path "/feda53ed-537d-4f88-9436-c6075776255b/f38b7023-3d53-43ea-b3db-e2c826d87b35" (reference "#PWR09") (unit 1)))))
 (wire (pts (xy 220.98 50.8) (xy 255.27 50.8)) (stroke (width 0) (type default)))
-(junction (at 220.98 50.8) (diameter 0) (color 0 0 0 0))
 (symbol (lib_id "power:GND") (at 255.27 58.42 0) (unit 1) (exclude_from_sim no) (in_bom no) (on_board no) (dnp no) (property "Reference" "#PWR10" (at 255.27 54.42 0) (effects (font (size 1.27 1.27)) (hide yes))) (property "Value" "GND" (at 255.27 62.23 0) (effects (font (size 1.27 1.27)))) (property "Footprint" "" (at 255.27 58.42 0) (effects (font (size 1.27 1.27)) (hide yes))) (property "Datasheet" "" (at 255.27 58.42 0) (effects (font (size 1.27 1.27)) (hide yes))) (pin "1") (instances (project "DesktopSpeaker" (path "/feda53ed-537d-4f88-9436-c6075776255b/f38b7023-3d53-43ea-b3db-e2c826d87b35" (reference "#PWR10") (unit 1)))))
 (wire (pts (xy 200.66 86.36) (xy 234.95 86.36)) (stroke (width 0) (type default)))

Commit message: Placement v9: EC11E volume encoder, 25 test points, silkscreen pass (closed sections, border, hole squares, labels), Orwellian logo on back, CAD refit
Co-Authored-By: Claude Sonnet 5.5 <noreply@anthropic.com>
Claude-Session: https://claude.ai/code/session_016fe4xPJbEE2SjGafuyNLjb
Parts:
- added TP1: USB_VBUS, DesktopSpeaker:TestPoint_Keystone_5015_Micro_Mini, symbol TestPoint:TestPoint
- added TP23: GND, DesktopSpeaker:TestPoint_Keystone_5010-5014_Multipurpose, symbol TestPoint:TestPoint
- added TP5: LDO_3V3, DesktopSpeaker:TestPoint_Keystone_5015_Micro_Mini, symbol TestPoint:TestPoint
Connections:
- net GND: now also TP23.1
- net LDO_3V3: now also TP5.1
- net USB_VBUS: now also TP1.1
Changed lines of the file:
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@@
 (symbol (lib_id "PD_PWR_FLAG:PD_PWR_FLAG") (at 114.3 71.12 270) (unit 1) (exclude_from_sim no) (in_bom no) (on_board no) (dnp no) (property "Reference" "#FLG303" (at 114.3 64.77000000000001 0) (effects (font (size 1.27 1.27)) (hide yes))) (property "Value" "PWR_FLAG" (at 114.3 67.31 0) (effects (font (size 1.27 1.27)) (hide yes))) (property "Footprint" "" (at 114.3 71.12 0) (hide yes) (effects (font (size 1.27 1.27)))) (property "Datasheet" "" (at 114.3 71.12 0) (hide yes) (effects (font (size 1.27 1.27)))) (pin "1") (instances (project "DesktopSpeaker" (path "/feda53ed-537d-4f88-9436-c6075776255b/f38b7023-3d53-43ea-b3db-e2c826d87b35" (reference "#FLG303") (unit 1)))))
 (wire (pts (xy 193.04 68.58) (xy 234.95 68.58)) (stroke (width 0) (type default)))
+(symbol (lib_id "TestPoint:TestPoint") (at 40.64 50.8 0) (unit 1) (exclude_from_sim no) (in_bom no) (on_board yes) (dnp no) (property "Reference" "TP1" (at 42.67 46.23 0) (effects (font (size 1.27 1.27)) (justify left))) (property "Value" "USB_VBUS" (at 42.67 48.77 0) (effects (font (size 1.27 1.27)) (justify left))) (property "Footprint" "DesktopSpeaker:TestPoint_Keystone_5015_Micro_Mini" (at 40.64 50.8 0) (hide yes) (effects (font (size 1.27 1.27)))) (property "Datasheet" "" (at 40.64 50.8 0) (hide yes) (effects (font (size 1.27 1.27)))) (property "Description" "Debug test point (excluded from BOM; hand-fitted loop)" (at 40.64 50.8 0) (hide yes) (effects (font (size 1 1)))) (pin "1") (instances (project "DesktopSpeaker" (path "/feda53ed-537d-4f88-9436-c6075776255b/f38b7023-3d53-43ea-b3db-e2c826d87b35" (reference "TP1") (unit 1)))))
+(wire (pts (xy 40.64 50.8) (xy 40.64 53.34)) (stroke (width 0) (type default)))
+(label "USB_VBUS" (at 40.64 53.34 0) (effects (font (size 1 1)) (justify left bottom)))
+(symbol (lib_id "TestPoint:TestPoint") (at 127 142.24 0) (unit 1) (exclude_from_sim no) (in_bom no) (on_board yes) (dnp no) (property "Reference" "TP5" (at 129.03 137.67 0) (effects (font (size 1.27 1.27)) (justify left))) (property "Value" "LDO_3V3" (at 129.03 140.21 0) (effects (font (size 1.27 1.27)) (justify left))) (property "Footprint" "DesktopSpeaker:TestPoint_Keystone_5015_Micro_Mini" (at 127 142.24 0) (hide yes) (effects (font (size 1.27 1.27)))) (property "Datasheet" "" (at 127 142.24 0) (hide yes) (effects (font (size 1.27 1.27)))) (property "Description" "Debug test point (excluded from BOM; hand-fitted loop)" (at 127 142.24 0) (hide yes) (effects (font (size 1 1)))) (pin "1") (instances (project "DesktopSpeaker" (path "/feda53ed-537d-4f88-9436-c6075776255b/f38b7023-3d53-43ea-b3db-e2c826d87b35" (reference "TP5") (unit 1)))))
+(wire (pts (xy 127 142.24) (xy 127 144.78)) (stroke (width 0) (type default)))
+(label "LDO_3V3" (at 127 144.78 0) (effects (font (size 1 1)) (justify left bottom)))
+(symbol (lib_id "TestPoint:TestPoint") (at 134.62 53.34 0) (unit 1) (exclude_from_sim no) (in_bom no) (on_board yes) (dnp no) (property "Reference" "TP23" (at 136.65 48.77 0) (effects (font (size 1.27 1.27)) (justify left))) (property "Value" "GND" (at 136.65 51.31 0) (effects (font (size 1.27 1.27)) (justify left))) (property "Footprint" "DesktopSpeaker:TestPoint_Keystone_5010-5014_Multipurpose" (at 134.62 53.34 0) (hide yes) (effects (font (size 1.27 1.27)))) (property "Datasheet" "" (at 134.62 53.34 0) (hide yes) (effects (font (size 1.27 1.27)))) (property "Description" "Debug test point (excluded from BOM; hand-fitted loop)" (at 134.62 53.34 0) (hide yes) (effects (font (size 1 1)))) (pin "1") (instances (project "DesktopSpeaker" (path "/feda53ed-537d-4f88-9436-c6075776255b/f38b7023-3d53-43ea-b3db-e2c826d87b35" (reference "TP23") (unit 1)))))
+(wire (pts (xy 134.62 53.34) (xy 134.62 55.88)) (stroke (width 0) (type default)))
+(symbol (lib_id "power:GND") (at 134.62 55.88 0) (unit 1) (exclude_from_sim no) (in_bom yes) (on_board no) (dnp no) (property "Reference" "#PWR1211" (at 134.62 59.69 0) (hide yes) (effects (font (size 1.27 1.27)))) (property "Value" "GND" (at 134.62 60.96 0) (hide yes) (effects (font (size 1.27 1.27)))) (pin "1") (instances (project "DesktopSpeaker" (path "/feda53ed-537d-4f88-9436-c6075776255b/f38b7023-3d53-43ea-b3db-e2c826d87b35" (reference "#PWR1211") (unit 1)))))
 )
