File: DesktopSpeaker-kicad/USB_PD.kicad_sch (KiCad schematic)
At the start: 25 parts, among them J4 I2C service, U11 TPS25730DREFR, U19 TPS7B8450QWDRBRQ1

Commit message: Schematic: add C311-C316, TP26/27; placement v10 to v10d (reviewed), reports and generators
Co-Authored-By: Claude Sonnet 5.5 <noreply@anthropic.com>
Claude-Session: https://claude.ai/code/session_016fe4xPJbEE2SjGafuyNLjb
Parts:
- added C315: 47uF 25V, DesktopSpeaker:PD_C_1206, symbol PD_C:PD_C
- added C316: 1uF X7R 50V, DesktopSpeaker:C_0805_2012Metric_Pad1.18x1.45mm_HandSolder, symbol PD_C:PD_C
Connections:
- net GND: now also C315.2, C316.2
- net USB_VBUS: now also C316.1
- net VBUS_PD: now also C315.1
Changed lines of the file:
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@@
 (wire (pts (xy 134.62 53.34) (xy 134.62 55.88)) (stroke (width 0) (type default)))
 (symbol (lib_id "power:GND") (at 134.62 55.88 0) (unit 1) (exclude_from_sim no) (in_bom yes) (on_board no) (dnp no) (property "Reference" "#PWR1211" (at 134.62 59.69 0) (hide yes) (effects (font (size 1.27 1.27)))) (property "Value" "GND" (at 134.62 60.96 0) (hide yes) (effects (font (size 1.27 1.27)))) (pin "1") (instances (project "DesktopSpeaker" (path "/feda53ed-537d-4f88-9436-c6075776255b/f38b7023-3d53-43ea-b3db-e2c826d87b35" (reference "#PWR1211") (unit 1)))))
-)
+(symbol (lib_id "PD_C:PD_C") (at 228.6 72.39 0) (unit 1) (exclude_from_sim no) (in_bom yes) (on_board yes) (dnp no) (property "Reference" "C315" (at 233.68 71.12 0) (effects (font (size 1.27 1.27)) (justify left))) (property "Value" "47uF 25V" (at 233.68 73.66 0) (effects (font (size 1.27 1.27)) (justify left))) (property "Footprint" "DesktopSpeaker:PD_C_1206" (at 228.6 72.39 0) (effects (font (size 1.0 1.0)) (hide yes))) (property "LCSC" "" (at 228.6 72.39 0) (hide yes) (effects (font (size 1 1)))) (property "Manufacturer" "Murata" (at 228.6 72.39 0) (effects (font (size 1.0 1.0)) (hide yes))) (property "MPN" "GRM31CR61E476ME44L" (at 228.6 72.39 0) (effects (font (size 1.0 1.0)) (hide yes))) (property "LCSC Part" "" (at 228.6 72.39 0) (effects (font (size 1.0 1.0)) (hide yes))) (property "Datasheet" "" (at 228.6 72.39 0) (effects (font (size 1.0 1.0)) (hide yes))) (pin "1") (pin "2") (instances (project "DesktopSpeaker" (path "/feda53ed-537d-4f88-9436-c6075776255b/f38b7023-3d53-43ea-b3db-e2c826d87b35" (reference "C315") (unit 1)))))
+(symbol (lib_id "power:GND") (at 228.6 76.2 0) (unit 1) (exclude_from_sim no) (in_bom no) (on_board no) (dnp no) (property "Reference" "#PWR2007" (at 233.68 74.93 0) (effects (font (size 1.27 1.27)) (justify left) (hide yes))) (property "Value" "GND" (at 228.6 81.28 0) (effects (font (size 1.27 1.27)))) (property "Footprint" "" (at 229.87 99.06 0) (effects (font (size 1.0 1.0)) (hide yes))) (pin "1") (instances (project "DesktopSpeaker" (path "/feda53ed-537d-4f88-9436-c6075776255b/f38b7023-3d53-43ea-b3db-e2c826d87b35" (reference "#PWR2007") (unit 1)))))
+(junction (at 228.6 68.58) (diameter 0) (color 0 0 0 0))
+(symbol (lib_id "PD_C:PD_C") (at 63.5 64.77 0) (unit 1) (exclude_from_sim no) (in_bom yes) (on_board yes) (dnp no) (property "Reference" "C316" (at 68.58 63.5 0) (effects (font (size 1.27 1.27)) (justify left))) (property "Value" "1uF X7R 50V" (at 68.58 66.04 0) (effects (font (size 1.27 1.27)) (justify left))) (property "Footprint" "DesktopSpeaker:C_0805_2012Metric_Pad1.18x1.45mm_HandSolder" (at 63.5 64.77 0) (effects (font (size 1.0 1.0)) (hide yes))) (property "LCSC" "" (at 63.5 64.77 0) (hide yes) (effects (font (size 1 1)))) (property "Manufacturer" "Samsung Electro-Mechanics" (at 63.5 64.77 0) (effects (font (size 1.0 1.0)) (hide yes))) (property "MPN" "CL21B105KBFNNNE" (at 63.5 64.77 0) (effects (font (size 1.0 1.0)) (hide yes))) (property "LCSC Part" "" (at 63.5 64.77 0) (effects (font (size 1.0 1.0)) (hide yes))) (property "Datasheet" "https://www.lcsc.com/datasheet/C28323.pdf" (at 63.5 64.77 0) (effects (font (size 1.0 1.0)) (hide yes))) (pin "1") (pin "2") (instances (project "DesktopSpeaker" (path "/feda53ed-537d-4f88-9436-c6075776255b/f38b7023-3d53-43ea-b3db-e2c826d87b35" (reference "C316") (unit 1)))))
+(symbol (lib_id "power:GND") (at 63.5 68.58 0) (unit 1) (exclude_from_sim no) (in_bom no) (on_board no) (dnp no) (property "Reference" "#PWR2008" (at 68.58 67.31 0) (effects (font (size 1.27 1.27)) (justify left) (hide yes))) (property "Value" "GND" (at 63.5 73.66 0) (effects (font (size 1.27 1.27)))) (property "Footprint" "" (at 64.77 91.44 0) (effects (font (size 1.0 1.0)) (hide yes))) (pin "1") (instances (project "DesktopSpeaker" (path "/feda53ed-537d-4f88-9436-c6075776255b/f38b7023-3d53-43ea-b3db-e2c826d87b35" (reference "#PWR2008") (unit 1)))))
+(junction (at 63.5 60.96) (diameter 0) (color 0 0 0 0)))

Commit message: Y200 24.576 MHz crystal with 15 pF load caps, C275 3D model, schematic/PCB sourcing fields synced to BOM
Co-Authored-By: Claude Sonnet 5.5 <noreply@anthropic.com>
Claude-Session: https://claude.ai/code/session_016fe4xPJbEE2SjGafuyNLjb
Parts:
- C182, C183: LCSC (none) -> C76965; LCSC Part (none) -> C76965
- C2: LCSC (none) -> C5159426; LCSC Part (none) -> C5159426; MPN C2012X7R1H475K125AC -> C2012X7R1H475KT0A0E
- C315: LCSC (none) -> C403725; LCSC Part (none) -> C403725
- C316: LCSC (none) -> C28323; LCSC Part (none) -> C28323
- C5: LCSC (none) -> C5159426; MPN C2012X7R1H475K125AC -> C2012X7R1H475KT0A0E
- D6: LCSC (none) -> C523793
- J4: LCSC (none) -> C124378; MPN (none) -> B-2100S04P-A110; Manufacturer (none) -> Ckmtw
- R10: LCSC (none) -> C114763; LCSC Part (none) -> C114763
