File: DesktopSpeaker-kicad/Amplifiers.kicad_sch (KiCad schematic)
At the start: 74 parts, among them J10 B2P-VH, J11 B2P-VH, J9 B2P-VH, U25 TPS61088RHLR, U6 TAS5825MRHBR, U7 TAS5825MRHBR

Commit message: Repackage passives to 0402/0805 hand-solder footprints; update BOM and flags
Co-Authored-By: Claude Sonnet 5.5 <noreply@anthropic.com>
Claude-Session: https://claude.ai/code/session_01N5RHheWSjDFDPbKVD5YVeJ
Parts:
- C260, C267, C276, C278, C281, C289, C291, C294: footprint DesktopSpeaker:PD_C_0603 -> DesktopSpeaker:C_0402_1005Metric_Pad0.74x0.62mm_HandSolder; LCSC C1591 -> C77020; MPN CL10B104KB8NNNC -> GRM155R71H104KE14D; Manufacturer Samsung Electro-Mechanics -> Murata
- C261, C262, C263, C264, C265, C270, C302, C303, C304, C305, C306, C307: footprint DesktopSpeaker:PD_C_0805 -> DesktopSpeaker:C_0805_2012Metric_Pad1.18x1.45mm_HandSolder
- C266: footprint DesktopSpeaker:PD_C_0603 -> DesktopSpeaker:C_0402_1005Metric_Pad0.74x0.62mm_HandSolder; LCSC C107093 -> (none); MPN CC0603KRX7R9BB473 -> GRM155R71H473KA12D; Manufacturer CCTC -> Murata
- C268: footprint DesktopSpeaker:PD_C_0603 -> DesktopSpeaker:C_0402_1005Metric_Pad0.74x0.62mm_HandSolder; MPN CL10B682KB8NNNC -> GRM155R71H682KA01D; Manufacturer Samsung Electro-Mechanics -> Murata
- C269: footprint DesktopSpeaker:PD_C_0603 -> DesktopSpeaker:C_0402_1005Metric_Pad0.74x0.62mm_HandSolder; MPN CL10C470JB8NNNC -> GRM1555C1H470JA01D; Manufacturer Samsung Electro-Mechanics -> Murata
- C271, C272, C273, C274, C277, C279, C290, C292: footprint DesktopSpeaker:PD_C_1210 -> DesktopSpeaker:C_0805_2012Metric_Pad1.18x1.45mm_HandSolder; LCSC C309062 -> (none); MPN CL32B226KAJNNNE -> CL21A226MAQNNNE
- C280, C293: footprint DesktopSpeaker:PD_C_0603 -> DesktopSpeaker:C_0805_2012Metric_Pad1.18x1.45mm_HandSolder; LCSC C19666 -> (none); MPN CL10A475KO8NNNC -> CL21A475KAQNNNE
- C282, C283, C284, C295, C296, C297: footprint DesktopSpeaker:PD_C_0805 -> DesktopSpeaker:C_0402_1005Metric_Pad0.74x0.62mm_HandSolder; LCSC C28323 -> C29266; MPN CL21B105KBFNNNE -> CL05A105KO5NNNC
- C285, C286, C287, C288, C298, C299, C300, C301: footprint DesktopSpeaker:PD_C_0603 -> DesktopSpeaker:C_0402_1005Metric_Pad0.74x0.62mm_HandSolder; MPN CL10B474KA8NNNC -> CL05B474KO5NNNC
- R250: footprint DesktopSpeaker:PD_R_0603 -> DesktopSpeaker:R_0402_1005Metric_Pad0.72x0.64mm_HandSolder; MPN RC0603FR-07499KL -> RC0402FR-07499KL; Manufacturer YAGEO -> Yageo
- R251: footprint DesktopSpeaker:PD_R_0603 -> DesktopSpeaker:R_0402_1005Metric_Pad0.72x0.64mm_HandSolder; MPN RC0603FR-0756KL -> RC0402FR-0756KL; Manufacturer YAGEO -> Yageo
- R252: footprint DesktopSpeaker:PD_R_0603 -> DesktopSpeaker:R_0402_1005Metric_Pad0.72x0.64mm_HandSolder; MPN RC0603FR-07301KL -> RC0402FR-07301KL; Manufacturer YAGEO -> Yageo
- R253: footprint DesktopSpeaker:PD_R_0603 -> DesktopSpeaker:R_0402_1005Metric_Pad0.72x0.64mm_HandSolder; MPN RC0603FR-07150KL -> RC0402FR-07150KL; Manufacturer YAGEO -> Yageo
- R254: footprint DesktopSpeaker:PD_R_0603 -> DesktopSpeaker:R_0402_1005Metric_Pad0.72x0.64mm_HandSolder; MPN RC0603FR-0782KL -> RC0402FR-0782KL; Manufacturer YAGEO -> Yageo
- R255, R259: footprint DesktopSpeaker:PD_R_0603 -> DesktopSpeaker:R_0402_1005Metric_Pad0.72x0.64mm_HandSolder; LCSC C14675 -> C60491; MPN RC0603FR-07100KL -> RC0402FR-07100KL; Manufacturer YAGEO -> Yageo
- R256, R260: footprint DesktopSpeaker:PD_R_0603 -> DesktopSpeaker:R_0402_1005Metric_Pad0.72x0.64mm_HandSolder; MPN RC0603FR-070RL -> RC0402FR-070RL; Manufacturer YAGEO -> Yageo
- R257, R258, R261: footprint DesktopSpeaker:PD_R_0603 -> DesktopSpeaker:R_0402_1005Metric_Pad0.72x0.64mm_HandSolder; LCSC C22548 -> (none); MPN RC0603FR-071KL -> RC0402FR-071KL; Manufacturer YAGEO -> Yageo
- R262: footprint DesktopSpeaker:PD_R_0603 -> DesktopSpeaker:R_0402_1005Metric_Pad0.72x0.64mm_HandSolder; LCSC C98220 -> C60490; MPN RC0603FR-0710KL -> RC0402FR-0710KL; Manufacturer YAGEO -> Yageo

Commit message: Apply low-risk passive cuts (11 parts) and normalise BOM; add layout rules and BOM audit reports
Co-Authored-By: Claude Sonnet 5.5 <noreply@anthropic.com>
Claude-Session: https://claude.ai/code/session_01N5RHheWSjDFDPbKVD5YVeJ
Parts:
- removed R260: 0R, DesktopSpeaker:R_0402_1005Metric_Pad0.72x0.64mm_HandSolder, symbol PD_R:PD_R
Connections:
- net GND: now also U6.8 (ADR)
Other:
- note added: "TAS5825M addresses: U6 ADR tied directly to GND = 0x4C, U7 ADR 1k = 0x4D. AMP_PDN shared (1k each, 100k pull-down). GPIO0 = FAULTZ (open drain) wired-OR to AMP_FAULT_N, 10k pull-up to 3V3_AUDIO. GPIO1/2 not connected."
- note removed: "TAS5825M addresses: U6 ADR 0R = 0x4C, U7 ADR 1k = 0x4D. AMP_PDN shared (1k each, 100k pull-down). GPIO0 = FAULTZ (open drain) wired-OR to AMP_FAULT_N, 10k pull-up to 3V3_AUDIO. GPIO1/2 not connected."
Changed lines of the file:
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@@
 (symbol (lib_id "PD_R:PD_R") (at 274.32 118.11 0) (unit 1) (exclude_from_sim no) (in_bom yes) (on_board yes) (dnp no) (property "Reference" "R259" (at 276.86 116.84 0) (effects (font (size 1.27 1.27)) (justify left))) (property "Value" "100k" (at 276.86 119.38 0) (effects (font (size 1.27 1.27)) (justify left))) (property "Footprint" "DesktopSpeaker:R_0402_1005Metric_Pad0.72x0.64mm_HandSolder" (at 274.32 118.11 0) (hide yes) (effects (font (size 1.27 1.27)))) (property "MPN" "RC0402FR-07100KL" (at 274.32 118.11 0) (hide yes) (effects (font (size 1.27 1.27)))) (property "Manufacturer" "Yageo" (at 274.32 118.11 0) (hide yes) (effects (font (size 1 1)))) (property "LCSC" "C60491" (at 274.32 118.11 0) (hide yes) (effects (font (size 1 1)))) (pin "1") (pin "2") (instances (project "DesktopSpeaker" (path "/feda53ed-537d-4f88-9436-c6075776255b/1c0e824e-98ce-4806-8137-f590f469c175" (reference "R259") (unit 1)))))
 (symbol (lib_id "power:GND") (at 274.32 121.92 0) (unit 1) (exclude_from_sim no) (in_bom no) (on_board no) (dnp no) (property "Reference" "#PWR1122" (at 274.32 125.73 0) (effects (font (size 1.27 1.27)) (hide yes))) (property "Value" "GND" (at 274.32 127 0) (effects (font (size 1.27 1.27)) (hide yes))) (pin "1") (instances (project "DesktopSpeaker" (path "/feda53ed-537d-4f88-9436-c6075776255b/1c0e824e-98ce-4806-8137-f590f469c175" (reference "#PWR1122") (unit 1)))))
-(symbol (lib_id "PD_R:PD_R") (at 290.83 121.92 90) (unit 1) (exclude_from_sim no) (in_bom yes) (on_board yes) (dnp no) (property "Reference" "R260" (at 290.83 117.22 270) (effects (font (size 1.27 1.27)) )) (property "Value" "0R" (at 290.83 118.72 270) (effects (font (size 1.27 1.27)) )) (property "Footprint" "DesktopSpeaker:R_0402_1005Metric_Pad0.72x0.64mm_HandSolder" (at 290.83 121.92 0) (hide yes) (effects (font (size 1.27 1.27)))) (property "MPN" "RC0402FR-070RL" (at 290.83 121.92 0) (hide yes) (effects (font (size 1.27 1.27)))) (property "Manufacturer" "Yageo" (at 290.83 121.92 0) (hide yes) (effects (font (size 1 1)))) (property "LCSC" "" (at 290.83 121.92 0) (hide yes) (effects (font (size 1 1)))) (pin "1") (pin "2") (instances (project "DesktopSpeaker" (path "/feda53ed-537d-4f88-9436-c6075776255b/1c0e824e-98ce-4806-8137-f590f469c175" (reference "R260") (unit 1)))))
-(symbol (lib_id "power:GND") (at 287.02 121.92 0) (unit 1) (exclude_from_sim no) (in_bom no) (on_board no) (dnp no) (property "Reference" "#PWR1123" (at 287.02 125.73 0) (effects (font (size 1.27 1.27)) (hide yes))) (property "Value" "GND" (at 287.02 127 0) (effects (font (size 1.27 1.27)) (hide yes))) (pin "1") (instances (project "DesktopSpeaker" (path "/feda53ed-537d-4f88-9436-c6075776255b/1c0e824e-98ce-4806-8137-f590f469c175" (reference "#PWR1123") (unit 1)))))
+(symbol (lib_id "power:GND") (at 294.64 121.92 0) (unit 1) (exclude_from_sim no) (in_bom no) (on_board no) (dnp no) (property "Reference" "#PWR1123" (at 294.64 125.73 0) (effects (font (size 1.27 1.27)) (hide yes))) (property "Value" "GND" (at 294.64 127 0) (effects (font (size 1.27 1.27)) (hide yes))) (pin "1") (instances (project "DesktopSpeaker" (path "/feda53ed-537d-4f88-9436-c6075776255b/1c0e824e-98ce-4806-8137-f590f469c175" (reference "#PWR1123") (unit 1)))))
 (wire (pts (xy 294.64 129.54) (xy 287.02 129.54)) (stroke (width 0) (type default)))
 (label "AMP_FAULT_N" (at 287.02 129.54 0) (effects (font (size 1 1)) (justify right bottom)))
@@
 (text "U25: VOUT = 1.204 V x (1 + 499k/56k) = 11.93 V (PFM: 12.0 V; OVP 12.7-13.6 V). FSW about 494 kHz (RFREQ 301k). ILIM 150k = 7.9 A typ, 6.6 A min in PFM (equation 3). L200 Isat 19.6 A." (at 40.64 231.14 0) (effects (font (size 1 1)) (justify left bottom)))
 (text "COMP: R254 82k, C268 6.8nF, C269 47pF (equations 18-20, fc about 5 kHz, effective Co about 170 uF): calculated only, bench check required. MODE floating = PFM; R256 DNP 0R to GND = forced PWM." (at 40.64 233.68 0) (effects (font (size 1 1)) (justify left bottom)))
-(text "TAS5825M addresses: U6 ADR 0R = 0x4C, U7 ADR 1k = 0x4D. AMP_PDN shared (1k each, 100k pull-down). GPIO0 = FAULTZ (open drain) wired-OR to AMP_FAULT_N, 10k pull-up to 3V3_AUDIO. GPIO1/2 not connected." (at 40.64 236.22 0) (effects (font (size 1 1)) (justify left bottom)))
+(text "TAS5825M addresses: U6 ADR tied directly to GND = 0x4C, U7 ADR 1k = 0x4D. AMP_PDN shared (1k each, 100k pull-down). GPIO0 = FAULTZ (open drain) wired-OR to AMP_FAULT_N, 10k pull-up to 3V3_AUDIO. GPIO1/2 not connected." (at 40.64 236.22 0) (effects (font (size 1 1)) (justify left bottom)))
 (text "DVDD = 3V3_AUDIO. Bootstrap caps are 0.47uF (Table 66). Filter 22uH + 0.68uF per output. No MCLK pin: TAS5825M locks to SCLK. Speaker connectors: pin 1 +, pin 2 -." (at 40.64 238.76 0) (effects (font (size 1 1)) (justify left bottom)))
 )

Commit message: Placement v9: EC11E volume encoder, 25 test points, silkscreen pass (closed sections, border, hole squares, labels), Orwellian logo on back, CAD refit
Co-Authored-By: Claude Sonnet 5.5 <noreply@anthropic.com>
Claude-Session: https://claude.ai/code/session_016fe4xPJbEE2SjGafuyNLjb
Parts:
- added TP10: PVDD_AMP, DesktopSpeaker:TestPoint_Keystone_5015_Micro_Mini, symbol TestPoint:TestPoint
- added TP20: AMP_FAULT_N, DesktopSpeaker:TestPoint_Keystone_5015_Micro_Mini, symbol TestPoint:TestPoint
- added TP24: GND, DesktopSpeaker:TestPoint_Keystone_5010-5014_Multipurpose, symbol TestPoint:TestPoint
Connections:
- net AMP_FAULT_N: now also TP20.1
- net GND: now also TP24.1
- net PVDD_AMP: now also TP10.1
Changed lines of the file:
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@@
 (text "TAS5825M addresses: U6 ADR tied directly to GND = 0x4C, U7 ADR 1k = 0x4D. AMP_PDN shared (1k each, 100k pull-down). GPIO0 = FAULTZ (open drain) wired-OR to AMP_FAULT_N, 10k pull-up to 3V3_AUDIO. GPIO1/2 not connected." (at 40.64 236.22 0) (effects (font (size 1 1)) (justify left bottom)))
 (text "DVDD = 3V3_AUDIO. Bootstrap caps are 0.47uF (Table 66). Filter 22uH + 0.68uF per output. No MCLK pin: TAS5825M locks to SCLK. Speaker connectors: pin 1 +, pin 2 -." (at 40.64 238.76 0) (effects (font (size 1 1)) (justify left bottom)))
+(symbol (lib_id "TestPoint:TestPoint") (at 254 142.24 0) (unit 1) (exclude_from_sim no) (in_bom no) (on_board yes) (dnp no) (property "Reference" "TP10" (at 256.03 137.67 0) (effects (font (size 1.27 1.27)) (justify left))) (property "Value" "PVDD_AMP" (at 256.03 140.21 0) (effects (font (size 1.27 1.27)) (justify left))) (property "Footprint" "DesktopSpeaker:TestPoint_Keystone_5015_Micro_Mini" (at 254 142.24 0) (hide yes) (effects (font (size 1.27 1.27)))) (property "Datasheet" "" (at 254 142.24 0) (hide yes) (effects (font (size 1.27 1.27)))) (property "Description" "Debug test point (excluded from BOM; hand-fitted loop)" (at 254 142.24 0) (hide yes) (effects (font (size 1 1)))) (pin "1") (instances (project "DesktopSpeaker" (path "/feda53ed-537d-4f88-9436-c6075776255b/1c0e824e-98ce-4806-8137-f590f469c175" (reference "TP10") (unit 1)))))
+(wire (pts (xy 254 142.24) (xy 254 144.78)) (stroke (width 0) (type default)))
+(label "PVDD_AMP" (at 254 144.78 0) (effects (font (size 1 1)) (justify left bottom)))
+(symbol (lib_id "TestPoint:TestPoint") (at 274.32 142.24 0) (unit 1) (exclude_from_sim no) (in_bom no) (on_board yes) (dnp no) (property "Reference" "TP20" (at 276.35 137.67 0) (effects (font (size 1.27 1.27)) (justify left))) (property "Value" "AMP_FAULT_N" (at 276.35 140.21 0) (effects (font (size 1.27 1.27)) (justify left))) (property "Footprint" "DesktopSpeaker:TestPoint_Keystone_5015_Micro_Mini" (at 274.32 142.24 0) (hide yes) (effects (font (size 1.27 1.27)))) (property "Datasheet" "" (at 274.32 142.24 0) (hide yes) (effects (font (size 1.27 1.27)))) (property "Description" "Debug test point (excluded from BOM; hand-fitted loop)" (at 274.32 142.24 0) (hide yes) (effects (font (size 1 1)))) (pin "1") (instances (project "DesktopSpeaker" (path "/feda53ed-537d-4f88-9436-c6075776255b/1c0e824e-98ce-4806-8137-f590f469c175" (reference "TP20") (unit 1)))))
+(wire (pts (xy 274.32 142.24) (xy 274.32 144.78)) (stroke (width 0) (type default)))
+(label "AMP_FAULT_N" (at 274.32 144.78 0) (effects (font (size 1 1)) (justify left bottom)))
+(symbol (lib_id "TestPoint:TestPoint") (at 114.3 127 0) (unit 1) (exclude_from_sim no) (in_bom no) (on_board yes) (dnp no) (property "Reference" "TP24" (at 116.33 122.43 0) (effects (font (size 1.27 1.27)) (justify left))) (property "Value" "GND" (at 116.33 124.97 0) (effects (font (size 1.27 1.27)) (justify left))) (property "Footprint" "DesktopSpeaker:TestPoint_Keystone_5010-5014_Multipurpose" (at 114.3 127 0) (hide yes) (effects (font (size 1.27 1.27)))) (property "Datasheet" "" (at 114.3 127 0) (hide yes) (effects (font (size 1.27 1.27)))) (property "Description" "Debug test point (excluded from BOM; hand-fitted loop)" (at 114.3 127 0) (hide yes) (effects (font (size 1 1)))) (pin "1") (instances (project "DesktopSpeaker" (path "/feda53ed-537d-4f88-9436-c6075776255b/1c0e824e-98ce-4806-8137-f590f469c175" (reference "TP24") (unit 1)))))
+(wire (pts (xy 114.3 127) (xy 114.3 129.54)) (stroke (width 0) (type default)))
+(symbol (lib_id "power:GND") (at 114.3 129.54 0) (unit 1) (exclude_from_sim no) (in_bom yes) (on_board no) (dnp no) (property "Reference" "#PWR1212" (at 114.3 133.35 0) (hide yes) (effects (font (size 1.27 1.27)))) (property "Value" "GND" (at 114.3 134.62 0) (hide yes) (effects (font (size 1.27 1.27)))) (pin "1") (instances (project "DesktopSpeaker" (path "/feda53ed-537d-4f88-9436-c6075776255b/1c0e824e-98ce-4806-8137-f590f469c175" (reference "#PWR1212") (unit 1)))))
 )

Commit message: Schematic: add C311-C316, TP26/27; placement v10 to v10d (reviewed), reports and generators
Co-Authored-By: Claude Sonnet 5.5 <noreply@anthropic.com>
Claude-Session: https://claude.ai/code/session_016fe4xPJbEE2SjGafuyNLjb
Parts:
- added C314: 100nF, DesktopSpeaker:C_0402_1005Metric_Pad0.74x0.62mm_HandSolder, symbol PD_C:PD_C
Connections:
- net GND: now also C314.2
- net PVDD_AMP: now also C314.1
Changed lines of the file:
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@@
 (wire (pts (xy 114.3 127) (xy 114.3 129.54)) (stroke (width 0) (type default)))
 (symbol (lib_id "power:GND") (at 114.3 129.54 0) (unit 1) (exclude_from_sim no) (in_bom yes) (on_board no) (dnp no) (property "Reference" "#PWR1212" (at 114.3 133.35 0) (hide yes) (effects (font (size 1.27 1.27)))) (property "Value" "GND" (at 114.3 134.62 0) (hide yes) (effects (font (size 1.27 1.27)))) (pin "1") (instances (project "DesktopSpeaker" (path "/feda53ed-537d-4f88-9436-c6075776255b/1c0e824e-98ce-4806-8137-f590f469c175" (reference "#PWR1212") (unit 1)))))
-)
+(symbol (lib_id "PD_C:PD_C") (at 266.7 153.67 0) (unit 1) (exclude_from_sim no) (in_bom yes) (on_board yes) (dnp no) (property "Reference" "C314" (at 271.78 152.4 0) (effects (font (size 1.27 1.27)) (justify left))) (property "Value" "100nF" (at 271.78 154.94 0) (effects (font (size 1.27 1.27)) (justify left))) (property "Footprint" "DesktopSpeaker:C_0402_1005Metric_Pad0.74x0.62mm_HandSolder" (at 266.7 153.67 0) (effects (font (size 1.0 1.0)) (hide yes))) (property "LCSC" "" (at 266.7 153.67 0) (hide yes) (effects (font (size 1 1)))) (property "Manufacturer" "Murata" (at 266.7 153.67 0) (effects (font (size 1.0 1.0)) (hide yes))) (property "MPN" "GRM155R71H104KE14D" (at 266.7 153.67 0) (effects (font (size 1.0 1.0)) (hide yes))) (property "LCSC Part" "" (at 266.7 153.67 0) (effects (font (size 1.0 1.0)) (hide yes))) (property "Datasheet" "${KIPRJMOD}/../ai-files/datasheets/Samsung_MLCC_LCSC_C1591_C1711.pdf" (at 266.7 153.67 0) (effects (font (size 1.0 1.0)) (hide yes))) (pin "1") (pin "2") (instances (project "DesktopSpeaker" (path "/feda53ed-537d-4f88-9436-c6075776255b/1c0e824e-98ce-4806-8137-f590f469c175" (reference "C314") (unit 1)))))
+(symbol (lib_id "power:GND") (at 266.7 157.48 0) (unit 1) (exclude_from_sim no) (in_bom no) (on_board no) (dnp no) (property "Reference" "#PWR2006" (at 271.78 156.21 0) (effects (font (size 1.27 1.27)) (justify left) (hide yes))) (property "Value" "GND" (at 266.7 162.56 0) (effects (font (size 1.27 1.27)))) (property "Footprint" "" (at 267.97 180.34 0) (effects (font (size 1.0 1.0)) (hide yes))) (pin "1") (instances (project "DesktopSpeaker" (path "/feda53ed-537d-4f88-9436-c6075776255b/1c0e824e-98ce-4806-8137-f590f469c175" (reference "#PWR2006") (unit 1)))))
+(wire (pts (xy 254 149.86) (xy 266.7 149.86)) (stroke (width 0) (type default))))

Commit message: Y200 24.576 MHz crystal with 15 pF load caps, C275 3D model, schematic/PCB sourcing fields synced to BOM
Co-Authored-By: Claude Sonnet 5.5 <noreply@anthropic.com>
Claude-Session: https://claude.ai/code/session_016fe4xPJbEE2SjGafuyNLjb
Parts:
- C266: LCSC (none) -> C117757; MPN GRM155R71H473KA12D -> GRM155R71H473KE14D
- C268: LCSC (none) -> C318580; MPN GRM155R71H682KA01D -> CL05B682KB5NNNC; Manufacturer Murata -> Samsung Electro-Mechanics
- C269: LCSC (none) -> C76970
- C271, C272, C273, C274, C277, C279, C290, C292: LCSC (none) -> C45783
- C275: LCSC (none) -> C264047; MPN EEH-ZA1E101P -> EEHZA1E101XP
- C280, C293: LCSC (none) -> C1779
- C285, C286, C287, C288, C298, C299, C300, C301: LCSC (none) -> C22435970; MPN CL05B474KO5NNNC -> CGA0402X7R474K160GT; Manufacturer Samsung Electro-Mechanics -> HRE
- C314: LCSC (none) -> C77020; LCSC Part (none) -> C77020
- L200: LCSC (none) -> C3911470
- L201, L202, L203, L204, L205, L206: LCSC (none) -> C7245133
- R250: LCSC (none) -> C137971
- R251: LCSC (none) -> C114756
- R252: LCSC (none) -> C171693
- R253: LCSC (none) -> C93947
- R254: LCSC (none) -> C144735; MPN RC0402FR-0782KL -> AC0402FR-0782KL
- R256: LCSC (none) -> C106231
- R257, R258, R261: LCSC (none) -> C106235
