File: DesktopSpeaker-kicad/Bluetooth.kicad_sch (KiCad schematic)
At the start: 16 parts, among them J8 BM83_PROG, U1 BM83SM1-00TA

Commit message: Repackage passives to 0402/0805 hand-solder footprints; update BOM and flags
Co-Authored-By: Claude Sonnet 5.5 <noreply@anthropic.com>
Claude-Session: https://claude.ai/code/session_01N5RHheWSjDFDPbKVD5YVeJ
Parts:
- C190: footprint DesktopSpeaker:PD_C_0805 -> DesktopSpeaker:C_0805_2012Metric_Pad1.18x1.45mm_HandSolder
- C191: footprint DesktopSpeaker:PD_C_0603 -> DesktopSpeaker:C_0402_1005Metric_Pad0.74x0.62mm_HandSolder; LCSC C1591 -> C77020; MPN CL10B104KB8NNNC -> GRM155R71H104KE14D; Manufacturer Samsung Electro-Mechanics -> Murata
- C192, C193: footprint DesktopSpeaker:PD_C_0805 -> DesktopSpeaker:C_0402_1005Metric_Pad0.74x0.62mm_HandSolder; LCSC C28323 -> C29266; MPN CL21B105KBFNNNE -> CL05A105KO5NNNC
- C194, C195: footprint DesktopSpeaker:PD_C_1206 -> DesktopSpeaker:C_0805_2012Metric_Pad1.18x1.45mm_HandSolder; LCSC C51205 -> (none); MPN CL31B475KBHNNNE -> CL21A475KAQNNNE
- R180, R181, R184: footprint DesktopSpeaker:PD_R_0603 -> DesktopSpeaker:R_0402_1005Metric_Pad0.72x0.64mm_HandSolder; LCSC C14675 -> C60491; MPN RC0603FR-07100KL -> RC0402FR-07100KL; Manufacturer YAGEO -> Yageo
- R182, R183: footprint DesktopSpeaker:PD_R_0603 -> DesktopSpeaker:R_0402_1005Metric_Pad0.72x0.64mm_HandSolder; LCSC C98220 -> C60490; MPN RC0603FR-0710KL -> RC0402FR-0710KL; Manufacturer YAGEO -> Yageo
- R185, R186, R187: footprint DesktopSpeaker:PD_R_0603 -> DesktopSpeaker:R_0402_1005Metric_Pad0.72x0.64mm_HandSolder; LCSC C22548 -> (none); MPN RC0603FR-071KL -> RC0402FR-071KL; Manufacturer YAGEO -> Yageo

Commit message: Placement v9: EC11E volume encoder, 25 test points, silkscreen pass (closed sections, border, hole squares, labels), Orwellian logo on back, CAD refit
Co-Authored-By: Claude Sonnet 5.5 <noreply@anthropic.com>
Claude-Session: https://claude.ai/code/session_016fe4xPJbEE2SjGafuyNLjb
Parts:
- added TP22: BT_UART_RX, DesktopSpeaker:TestPoint_Keystone_5015_Micro_Mini, symbol TestPoint:TestPoint
Connections:
- net BT_UART_RX: now also TP22.1
Changed lines of the file:
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@@
 (text "Antenna: integrated PCB antenna, no external RF parts. Keep the antenna end of the module off the board (no copper/components/keep-out) and metal 15 mm clear; see ai-files/reports/bluetooth-notes.md." (at 77.47 182.3 0) (effects (font (size 1 1)) (justify left bottom)))
 (text "J8 programming/test (isUpdate/Config Tool): 1 RST_N, 2 P3_4 SYS_CFG (low at reset = test mode), 3 UART_RXD (adapter TX), 4 UART_TXD (adapter RX), 5 GND. 3V8_BT must be enabled first." (at 77.47 185.3 0) (effects (font (size 1 1)) (justify left bottom)))
+(symbol (lib_id "TestPoint:TestPoint") (at 223.52 81.28 0) (unit 1) (exclude_from_sim no) (in_bom no) (on_board yes) (dnp no) (property "Reference" "TP22" (at 225.55 76.71 0) (effects (font (size 1.27 1.27)) (justify left))) (property "Value" "BT_UART_RX" (at 225.55 79.25 0) (effects (font (size 1.27 1.27)) (justify left))) (property "Footprint" "DesktopSpeaker:TestPoint_Keystone_5015_Micro_Mini" (at 223.52 81.28 0) (hide yes) (effects (font (size 1.27 1.27)))) (property "Datasheet" "" (at 223.52 81.28 0) (hide yes) (effects (font (size 1.27 1.27)))) (property "Description" "Debug test point (excluded from BOM; hand-fitted loop)" (at 223.52 81.28 0) (hide yes) (effects (font (size 1 1)))) (pin "1") (instances (project "DesktopSpeaker" (path "/feda53ed-537d-4f88-9436-c6075776255b/cc34ef9a-e98e-4641-98b8-a2a9303b711c" (reference "TP22") (unit 1)))))
+(wire (pts (xy 223.52 81.28) (xy 223.52 83.82)) (stroke (width 0) (type default)))
+(label "BT_UART_RX" (at 223.52 83.82 0) (effects (font (size 1 1)) (justify left bottom)))
 )

Commit message: Y200 24.576 MHz crystal with 15 pF load caps, C275 3D model, schematic/PCB sourcing fields synced to BOM
Co-Authored-By: Claude Sonnet 5.5 <noreply@anthropic.com>
Claude-Session: https://claude.ai/code/session_016fe4xPJbEE2SjGafuyNLjb
Parts:
- C194, C195: LCSC (none) -> C1779
- R185, R186, R187: LCSC (none) -> C106235
