File: DesktopSpeaker-kicad/Bluetooth_Power.kicad_sch (KiCad schematic)
At the start: 12 parts, among them U15 TPS63802DLAR

Commit message: Repackage passives to 0402/0805 hand-solder footprints; update BOM and flags
Co-Authored-By: Claude Sonnet 5.5 <noreply@anthropic.com>
Claude-Session: https://claude.ai/code/session_01N5RHheWSjDFDPbKVD5YVeJ
Parts:
- C150, C152, C153, C154: footprint DesktopSpeaker:PD_C_0805 -> DesktopSpeaker:C_0805_2012Metric_Pad1.18x1.45mm_HandSolder; LCSC (none) -> C907991; Manufacturer (none) -> Murata
- C151: footprint DesktopSpeaker:PD_C_0603 -> DesktopSpeaker:C_0402_1005Metric_Pad0.74x0.62mm_HandSolder; LCSC C1591 -> C77020; LCSC Part C1591 -> C77020; MPN CL10B104KB8NNNC -> GRM155R71H104KE14D; Manufacturer Samsung Electro-Mechanics -> Murata
- R150: footprint DesktopSpeaker:PD_R_0603 -> DesktopSpeaker:R_0402_1005Metric_Pad0.72x0.64mm_HandSolder; LCSC C2933246 -> (none); MPN FRC0603F6043TS -> RC0402FR-07604KL; Manufacturer FOJAN -> Yageo
- R151: footprint DesktopSpeaker:PD_R_0603 -> DesktopSpeaker:R_0402_1005Metric_Pad0.72x0.64mm_HandSolder; LCSC C228098 -> (none); MPN AC0603FR-0791KL -> RC0402FR-0791KL; Manufacturer YAGEO -> Yageo
- R152, R153, R154: footprint DesktopSpeaker:PD_R_0603 -> DesktopSpeaker:R_0402_1005Metric_Pad0.72x0.64mm_HandSolder; LCSC C14675 -> C60491; MPN RC0603FR-07100KL -> RC0402FR-07100KL; Manufacturer YAGEO -> Yageo

Commit message: Apply low-risk passive cuts (11 parts) and normalise BOM; add layout rules and BOM audit reports
Co-Authored-By: Claude Sonnet 5.5 <noreply@anthropic.com>
Claude-Session: https://claude.ai/code/session_01N5RHheWSjDFDPbKVD5YVeJ
Parts:
- removed C151: 100nF 10V X7R, DesktopSpeaker:C_0402_1005Metric_Pad0.74x0.62mm_HandSolder, symbol PD_C:PD_C

Commit message: Placement v9: EC11E volume encoder, 25 test points, silkscreen pass (closed sections, border, hole squares, labels), Orwellian logo on back, CAD refit
Co-Authored-By: Claude Sonnet 5.5 <noreply@anthropic.com>
Claude-Session: https://claude.ai/code/session_016fe4xPJbEE2SjGafuyNLjb
Parts:
- added TP9: 3V8_BT, DesktopSpeaker:TestPoint_Keystone_5015_Micro_Mini, symbol TestPoint:TestPoint
Connections:
- net 3V8_BT: now also TP9.1

Commit message: Y200 24.576 MHz crystal with 15 pF load caps, C275 3D model, schematic/PCB sourcing fields synced to BOM
Co-Authored-By: Claude Sonnet 5.5 <noreply@anthropic.com>
Claude-Session: https://claude.ai/code/session_016fe4xPJbEE2SjGafuyNLjb
Parts:
- L3: Manufacturer (none) -> Coilcraft
- R150: LCSC (none) -> C27013; MPN RC0402FR-07604KL -> 0402WGF6043TCE; Manufacturer Yageo -> UNI-ROYAL
- R151: LCSC (none) -> C144733; MPN RC0402FR-0791KL -> AC0402FR-0791KL
- U15: Manufacturer (none) -> Texas Instruments
