File: DesktopSpeaker-kicad/Fuel_Gauge_Power.kicad_sch (KiCad schematic)
At the start: 25 parts, among them Q104 2N7002, U12 TPS7A0230PDBVR, U13 TS5A3167DBVR, U16 TS5A3167DBVR, U17 TS5A3167DBVR, U20 TPS2116DRLR, U21 TPS3839G33DBZR, U5 MAX17048G+T10

Commit message: Repackage passives to 0402/0805 hand-solder footprints; update BOM and flags
Co-Authored-By: Claude Sonnet 5.5 <noreply@anthropic.com>
Claude-Session: https://claude.ai/code/session_01N5RHheWSjDFDPbKVD5YVeJ
Parts:
- C120, C121, C126, C130, C131, C132: footprint DesktopSpeaker:PD_C_0603 -> DesktopSpeaker:C_0402_1005Metric_Pad0.74x0.62mm_HandSolder; LCSC C1591 -> C77020; MPN CL10B104KB8NNNC -> GRM155R71H104KE14D; Manufacturer Samsung Electro-Mechanics -> Murata
- C122, C123, C124, C125: value 1uF X7R 10V -> 1uF X5R 16V; footprint DesktopSpeaker:PD_C_0603 -> DesktopSpeaker:C_0402_1005Metric_Pad0.74x0.62mm_HandSolder; LCSC C92806 -> C29266; MPN LMK107B7105KA-T -> CL05A105KO5NNNC; Manufacturer Taiyo Yuden -> Samsung Electro-Mechanics
- R120, R121: footprint DesktopSpeaker:PD_R_0603 -> DesktopSpeaker:R_0402_1005Metric_Pad0.72x0.64mm_HandSolder; LCSC C99782 -> (none); MPN RC0603FR-074K7L -> RC0402FR-074K7L; Manufacturer YAGEO -> Yageo
- R122: footprint DesktopSpeaker:PD_R_0603 -> DesktopSpeaker:R_0402_1005Metric_Pad0.72x0.64mm_HandSolder; LCSC C105579 -> (none); MPN RC0603FR-0747KL -> RC0402FR-0747KL; Manufacturer YAGEO -> Yageo
- R124: footprint DesktopSpeaker:PD_R_0603 -> DesktopSpeaker:R_0402_1005Metric_Pad0.72x0.64mm_HandSolder; LCSC C123419 -> (none); LCSC Part C123419 -> (none); MPN RC0603FR-07180KL -> RC0402FR-07180KL
- R125: footprint DesktopSpeaker:PD_R_0603 -> DesktopSpeaker:R_0402_1005Metric_Pad0.72x0.64mm_HandSolder; LCSC C14675 -> C60491; LCSC Part C14675 -> C60491; MPN RC0603FR-07100KL -> RC0402FR-07100KL
- R126, R127: footprint DesktopSpeaker:PD_R_0603 -> DesktopSpeaker:R_0402_1005Metric_Pad0.72x0.64mm_HandSolder; LCSC C105578 -> (none); MPN RC0603FR-071ML -> RC0402FR-071ML; Manufacturer YAGEO -> Yageo

Commit message: Apply low-risk passive cuts (11 parts) and normalise BOM; add layout rules and BOM audit reports
Co-Authored-By: Claude Sonnet 5.5 <noreply@anthropic.com>
Claude-Session: https://claude.ai/code/session_01N5RHheWSjDFDPbKVD5YVeJ
Parts:
- removed C121: 100nF X7R 10V, DesktopSpeaker:C_0402_1005Metric_Pad0.74x0.62mm_HandSolder, symbol PD_C:PD_C
Changed lines of the file:
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@@
 (wire (pts (xy 35.56 73.66) (xy 120.65 73.66)) (stroke (width 0) (type default)))
 (wire (pts (xy 120.65 73.66) (xy 146.05 73.66)) (stroke (width 0) (type default)))
-(wire (pts (xy 146.05 73.66) (xy 177.8 73.66)) (stroke (width 0) (type default)))
 (wire (pts (xy 146.05 73.66) (xy 146.05 109.22)) (stroke (width 0) (type default)))
 (wire (pts (xy 146.05 109.22) (xy 165.1 109.22)) (stroke (width 0) (type default)))
-(junction (at 146.05 73.66) (diameter 0) (color 0 0 0 0))
 (symbol (lib_id "PD_C:PD_C") (at 120.65 88.9 0) (unit 1) (exclude_from_sim no) (in_bom yes) (on_board yes) (dnp no) (property "Reference" "C120" (at 124.65 87.63 0) (effects (font (size 1.27 1.27)) (justify left))) (property "Value" "100nF X7R 10V" (at 124.65 90.17 0) (effects (font (size 1.27 1.27)) (justify left))) (property "Footprint" "DesktopSpeaker:C_0402_1005Metric_Pad0.74x0.62mm_HandSolder" (at 120.65 88.9 0) (hide yes) (effects (font (size 1.27 1.27)))) (property "Datasheet" "${KIPRJMOD}/../ai-files/datasheets/Samsung_MLCC_LCSC_C1591_C1711.pdf" (at 120.65 88.9 0) (hide yes) (effects (font (size 1.27 1.27)))) (property "MPN" "GRM155R71H104KE14D" (at 120.65 88.9 0) (hide yes) (effects (font (size 1.27 1.27)))) (pin "1") (pin "2") (instances (project "DesktopSpeaker" (path "/feda53ed-537d-4f88-9436-c6075776255b/9c37a727-9991-421a-8f6e-77dd39bb53fa" (reference "C120") (unit 1)))) (property "Manufacturer" "Murata" (at 120.65 88.9 0) (effects (font (size 1 1)) (hide yes))) (property "LCSC" "C77020" (at 120.65 88.9 0) (effects (font (size 1 1)) (hide yes))))
 (wire (pts (xy 120.65 73.66) (xy 120.65 85.09)) (stroke (width 0) (type default)))
@@
 (wire (pts (xy 190.5 109.22) (xy 198.12 109.22)) (stroke (width 0) (type default)))
 (symbol (lib_id "power:GND") (at 198.12 109.22 0) (unit 1) (exclude_from_sim no) (in_bom no) (on_board no) (dnp no) (property "Reference" "#PWR108" (at 198.12 113.03 0) (effects (font (size 1.27 1.27)) (hide yes))) (property "Value" "GND" (at 198.12 114.3 0) (effects (font (size 1.27 1.27)))) (pin "1") (instances (project "DesktopSpeaker" (path "/feda53ed-537d-4f88-9436-c6075776255b/9c37a727-9991-421a-8f6e-77dd39bb53fa" (reference "#PWR108") (unit 1)))))
-(symbol (lib_id "PD_C:PD_C") (at 177.8 81.28 0) (unit 1) (exclude_from_sim no) (in_bom yes) (on_board yes) (dnp no) (property "Reference" "C121" (at 181.8 80.01 0) (effects (font (size 1.27 1.27)) (justify left))) (property "Value" "100nF X7R 10V" (at 181.8 82.55 0) (effects (font (size 1.27 1.27)) (justify left))) (property "Footprint" "DesktopSpeaker:C_0402_1005Metric_Pad0.74x0.62mm_HandSolder" (at 177.8 81.28 0) (hide yes) (effects (font (size 1.27 1.27)))) (property "Datasheet" "${KIPRJMOD}/../ai-files/datasheets/Samsung_MLCC_LCSC_C1591_C1711.pdf" (at 177.8 81.28 0) (hide yes) (effects (font (size 1.27 1.27)))) (property "MPN" "GRM155R71H104KE14D" (at 177.8 81.28 0) (hide yes) (effects (font (size 1.27 1.27)))) (pin "1") (pin "2") (instances (project "DesktopSpeaker" (path "/feda53ed-537d-4f88-9436-c6075776255b/9c37a727-9991-421a-8f6e-77dd39bb53fa" (reference "C121") (unit 1)))) (property "Manufacturer" "Murata" (at 177.8 81.28 0) (effects (font (size 1 1)) (hide yes))) (property "LCSC" "C77020" (at 177.8 81.28 0) (effects (font (size 1 1)) (hide yes))))
-(wire (pts (xy 177.8 73.66) (xy 177.8 77.47)) (stroke (width 0) (type default)))
-(junction (at 177.8 73.66) (diameter 0) (color 0 0 0 0))
-(wire (pts (xy 177.8 85.09) (xy 177.8 90.17)) (stroke (width 0) (type default)))
-(symbol (lib_id "power:GND") (at 177.8 90.17 0) (unit 1) (exclude_from_sim no) (in_bom no) (on_board no) (dnp no) (property "Reference" "#PWR109" (at 177.8 93.98 0) (effects (font (size 1.27 1.27)) (hide yes))) (property "Value" "GND" (at 177.8 95.25 0) (effects (font (size 1.27 1.27)))) (pin "1") (instances (project "DesktopSpeaker" (path "/feda53ed-537d-4f88-9436-c6075776255b/9c37a727-9991-421a-8f6e-77dd39bb53fa" (reference "#PWR109") (unit 1)))))
 (hierarchical_label "GAUGE_SCL" (shape input) (at 35.56 146.05 0) (effects (font (size 1.0 1.0)) (justify left bottom)))
 (hierarchical_label "GAUGE_SDA" (shape bidirectional) (at 35.56 151.13 0) (effects (font (size 1.0 1.0)) (justify left bottom)))

Commit message: Placement v9: EC11E volume encoder, 25 test points, silkscreen pass (closed sections, border, hole squares, labels), Orwellian logo on back, CAD refit
Co-Authored-By: Claude Sonnet 5.5 <noreply@anthropic.com>
Claude-Session: https://claude.ai/code/session_016fe4xPJbEE2SjGafuyNLjb
Parts:
- added TP3: BAT_PACK, DesktopSpeaker:TestPoint_Keystone_5015_Micro_Mini, symbol TestPoint:TestPoint
- added TP4: 3V_AO, DesktopSpeaker:TestPoint_Keystone_5015_Micro_Mini, symbol TestPoint:TestPoint
Connections:
- net 3V_AO: now also TP4.1
- net BAT_PACK: now also TP3.1
Changed lines of the file:
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@@
 (wire (pts (xy 96.52 119.38) (xy 88.9 119.38)) (stroke (width 0) (type default)))
 (wire (pts (xy 88.9 119.38) (xy 88.9 128.27)) (stroke (width 0) (type default)))
+(symbol (lib_id "TestPoint:TestPoint") (at 35.56 83.82 0) (unit 1) (exclude_from_sim no) (in_bom no) (on_board yes) (dnp no) (property "Reference" "TP3" (at 37.59 79.25 0) (effects (font (size 1.27 1.27)) (justify left))) (property "Value" "BAT_PACK" (at 37.59 81.79 0) (effects (font (size 1.27 1.27)) (justify left))) (property "Footprint" "DesktopSpeaker:TestPoint_Keystone_5015_Micro_Mini" (at 35.56 83.82 0) (hide yes) (effects (font (size 1.27 1.27)))) (property "Datasheet" "" (at 35.56 83.82 0) (hide yes) (effects (font (size 1.27 1.27)))) (property "Description" "Debug test point (excluded from BOM; hand-fitted loop)" (at 35.56 83.82 0) (hide yes) (effects (font (size 1 1)))) (pin "1") (instances (project "DesktopSpeaker" (path "/feda53ed-537d-4f88-9436-c6075776255b/9c37a727-9991-421a-8f6e-77dd39bb53fa" (reference "TP3") (unit 1)))))
+(wire (pts (xy 35.56 83.82) (xy 35.56 86.36)) (stroke (width 0) (type default)))
+(label "BAT_PACK" (at 35.56 86.36 0) (effects (font (size 1 1)) (justify left bottom)))
+(symbol (lib_id "TestPoint:TestPoint") (at 271.78 20.32 0) (unit 1) (exclude_from_sim no) (in_bom no) (on_board yes) (dnp no) (property "Reference" "TP4" (at 273.81 15.75 0) (effects (font (size 1.27 1.27)) (justify left))) (property "Value" "3V_AO" (at 273.81 18.29 0) (effects (font (size 1.27 1.27)) (justify left))) (property "Footprint" "DesktopSpeaker:TestPoint_Keystone_5015_Micro_Mini" (at 271.78 20.32 0) (hide yes) (effects (font (size 1.27 1.27)))) (property "Datasheet" "" (at 271.78 20.32 0) (hide yes) (effects (font (size 1.27 1.27)))) (property "Description" "Debug test point (excluded from BOM; hand-fitted loop)" (at 271.78 20.32 0) (hide yes) (effects (font (size 1 1)))) (pin "1") (instances (project "DesktopSpeaker" (path "/feda53ed-537d-4f88-9436-c6075776255b/9c37a727-9991-421a-8f6e-77dd39bb53fa" (reference "TP4") (unit 1)))))
+(wire (pts (xy 271.78 20.32) (xy 271.78 22.86)) (stroke (width 0) (type default)))
+(label "3V_AO" (at 271.78 22.86 0) (effects (font (size 1 1)) (justify left bottom)))
 )

Commit message: Y200 24.576 MHz crystal with 15 pF load caps, C275 3D model, schematic/PCB sourcing fields synced to BOM
Co-Authored-By: Claude Sonnet 5.5 <noreply@anthropic.com>
Claude-Session: https://claude.ai/code/session_016fe4xPJbEE2SjGafuyNLjb
Parts:
- R120, R121: LCSC (none) -> C105871
- R122: LCSC (none) -> C93943
- R124: LCSC (none) -> C138046; LCSC Part (none) -> C138046
- R126, R127: LCSC (none) -> C138033
- U12, U13, U16, U17: Manufacturer (none) -> Texas Instruments
