File: DesktopSpeaker-kicad/Headphone_Aux.kicad_sch (KiCad schematic)
At the start: 49 parts, among them J2 HEAD_OUT, J3 AUX_IN, U10 TPA6132A2RTER, U8 TS5A23157DGSR, U9 TS5A23157DGSR

Commit message: Repackage passives to 0402/0805 hand-solder footprints; update BOM and flags
Co-Authored-By: Claude Sonnet 5.5 <noreply@anthropic.com>
Claude-Session: https://claude.ai/code/session_01N5RHheWSjDFDPbKVD5YVeJ
Parts:
- C230, C231, C232, C233, C234, C235, C239, C240, C241, C245: footprint DesktopSpeaker:PD_C_0805 -> DesktopSpeaker:C_0402_1005Metric_Pad0.74x0.62mm_HandSolder; LCSC C28323 -> C29266; MPN CL21B105KBFNNNE -> CL05A105KO5NNNC
- C236: footprint DesktopSpeaker:PD_C_1206 -> DesktopSpeaker:C_0805_2012Metric_Pad1.18x1.45mm_HandSolder; LCSC C51205 -> (none); MPN CL31B475KBHNNNE -> CL21A475KAQNNNE
- C237, C238, C242, C246: footprint DesktopSpeaker:PD_C_0603 -> DesktopSpeaker:C_0402_1005Metric_Pad0.74x0.62mm_HandSolder; LCSC C1591 -> C77020; MPN CL10B104KB8NNNC -> GRM155R71H104KE14D; Manufacturer Samsung Electro-Mechanics -> Murata
- C243, C244: footprint DesktopSpeaker:PD_C_0805 -> DesktopSpeaker:C_0402_1005Metric_Pad0.74x0.62mm_HandSolder; LCSC C19110 -> (none); MPN CL21B225KAFNNNE -> CL05A225KP5NNNC
- R220, R221, R222, R223, R224, R225, R234, R235, R236, R237, R238, R239: footprint DesktopSpeaker:PD_R_0603 -> DesktopSpeaker:R_0402_1005Metric_Pad0.72x0.64mm_HandSolder; LCSC C14675 -> C60491; MPN RC0603FR-07100KL -> RC0402FR-07100KL; Manufacturer YAGEO -> Yageo
- R226, R227, R228, R229, R230, R231, R240: footprint DesktopSpeaker:PD_R_0603 -> DesktopSpeaker:R_0402_1005Metric_Pad0.72x0.64mm_HandSolder; LCSC C22548 -> (none); MPN RC0603FR-071KL -> RC0402FR-071KL; Manufacturer YAGEO -> Yageo
- R232, R233: footprint DesktopSpeaker:PD_R_0603 -> DesktopSpeaker:R_0402_1005Metric_Pad0.72x0.64mm_HandSolder; LCSC C105579 -> (none); MPN RC0603FR-0747KL -> RC0402FR-0747KL; Manufacturer YAGEO -> Yageo
- R241: footprint DesktopSpeaker:PD_R_0603 -> DesktopSpeaker:R_0402_1005Metric_Pad0.72x0.64mm_HandSolder; LCSC C105578 -> (none); MPN RC0603FR-071ML -> RC0402FR-071ML; Manufacturer YAGEO -> Yageo
- R242, R243, R244: footprint DesktopSpeaker:PD_R_0603 -> DesktopSpeaker:R_0402_1005Metric_Pad0.72x0.64mm_HandSolder; LCSC C98220 -> C60490; MPN RC0603FR-0710KL -> RC0402FR-0710KL; Manufacturer YAGEO -> Yageo

Commit message: Apply low-risk passive cuts (11 parts) and normalise BOM; add layout rules and BOM audit reports
Co-Authored-By: Claude Sonnet 5.5 <noreply@anthropic.com>
Claude-Session: https://claude.ai/code/session_01N5RHheWSjDFDPbKVD5YVeJ
Parts:
- removed C242: 100nF, DesktopSpeaker:C_0402_1005Metric_Pad0.74x0.62mm_HandSolder, symbol PD_C:PD_C
Changed lines of the file:
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@@
 (label "HP_G1" (at 259.08 128.27 0) (effects (font (size 1 1)) (justify right bottom)))
 (wire (pts (xy 271.78 92.71) (xy 271.78 80.01)) (stroke (width 0) (type default)))
-(wire (pts (xy 271.78 80.01) (xy 256.54 80.01)) (stroke (width 0) (type default)))
+(wire (pts (xy 271.78 80.01) (xy 264.16 80.01)) (stroke (width 0) (type default)))
 (label "3V3_AUDIO" (at 271.78 80.01 0) (effects (font (size 1 1)) (justify left bottom)))
-(junction (at 264.16 80.01) (diameter 0) (color 0 0 0 0))
 (symbol (lib_id "PD_C:PD_C") (at 264.16 83.82 0) (unit 1) (exclude_from_sim no) (in_bom yes) (on_board yes) (dnp no) (property "Reference" "C241" (at 265.43 82.55 0) (effects (font (size 1.27 1.27)) (justify left))) (property "Value" "1uF" (at 265.43 85.09 0) (effects (font (size 1.27 1.27)) (justify left))) (property "Footprint" "DesktopSpeaker:C_0402_1005Metric_Pad0.74x0.62mm_HandSolder" (at 264.16 83.82 0) (hide yes) (effects (font (size 1.27 1.27)))) (property "MPN" "CL05A105KO5NNNC" (at 264.16 83.82 0) (hide yes) (effects (font (size 1.27 1.27)))) (property "Manufacturer" "Samsung Electro-Mechanics" (at 264.16 83.82 0) (hide yes) (effects (font (size 1 1)))) (property "LCSC" "C29266" (at 264.16 83.82 0) (hide yes) (effects (font (size 1 1)))) (pin "1") (pin "2") (instances (project "DesktopSpeaker" (path "/feda53ed-537d-4f88-9436-c6075776255b/07901b33-a7e7-4327-b949-fc2abc1e14b5" (reference "C241") (unit 1)))))
 (symbol (lib_id "power:GND") (at 264.16 87.63 0) (unit 1) (exclude_from_sim no) (in_bom no) (on_board no) (dnp no) (property "Reference" "#PWR1005" (at 264.16 91.44 0) (effects (font (size 1.27 1.27)) (hide yes))) (property "Value" "GND" (at 264.16 92.71 0) (effects (font (size 1.27 1.27)) (hide yes))) (pin "1") (instances (project "DesktopSpeaker" (path "/feda53ed-537d-4f88-9436-c6075776255b/07901b33-a7e7-4327-b949-fc2abc1e14b5" (reference "#PWR1005") (unit 1)))))
-(symbol (lib_id "PD_C:PD_C") (at 256.54 83.82 0) (unit 1) (exclude_from_sim no) (in_bom yes) (on_board yes) (dnp no) (property "Reference" "C242" (at 257.81 82.55 0) (effects (font (size 1.27 1.27)) (justify left))) (property "Value" "100nF" (at 257.81 85.09 0) (effects (font (size 1.27 1.27)) (justify left))) (property "Footprint" "DesktopSpeaker:C_0402_1005Metric_Pad0.74x0.62mm_HandSolder" (at 256.54 83.82 0) (hide yes) (effects (font (size 1.27 1.27)))) (property "MPN" "GRM155R71H104KE14D" (at 256.54 83.82 0) (hide yes) (effects (font (size 1.27 1.27)))) (property "Manufacturer" "Murata" (at 256.54 83.82 0) (hide yes) (effects (font (size 1 1)))) (property "LCSC" "C77020" (at 256.54 83.82 0) (hide yes) (effects (font (size 1 1)))) (pin "1") (pin "2") (instances (project "DesktopSpeaker" (path "/feda53ed-537d-4f88-9436-c6075776255b/07901b33-a7e7-4327-b949-fc2abc1e14b5" (reference "C242") (unit 1)))))
-(symbol (lib_id "power:GND") (at 256.54 87.63 0) (unit 1) (exclude_from_sim no) (in_bom no) (on_board no) (dnp no) (property "Reference" "#PWR1006" (at 256.54 91.44 0) (effects (font (size 1.27 1.27)) (hide yes))) (property "Value" "GND" (at 256.54 92.71 0) (effects (font (size 1.27 1.27)) (hide yes))) (pin "1") (instances (project "DesktopSpeaker" (path "/feda53ed-537d-4f88-9436-c6075776255b/07901b33-a7e7-4327-b949-fc2abc1e14b5" (reference "#PWR1006") (unit 1)))))
 (symbol (lib_id "power:GND") (at 269.24 146.05 0) (unit 1) (exclude_from_sim no) (in_bom no) (on_board no) (dnp no) (property "Reference" "#PWR1007" (at 269.24 149.86 0) (effects (font (size 1.27 1.27)) (hide yes))) (property "Value" "GND" (at 269.24 151.13 0) (effects (font (size 1.27 1.27)) (hide yes))) (pin "1") (instances (project "DesktopSpeaker" (path "/feda53ed-537d-4f88-9436-c6075776255b/07901b33-a7e7-4327-b949-fc2abc1e14b5" (reference "#PWR1007") (unit 1)))))
 (wire (pts (xy 297.18 118.11) (xy 300.99 118.11)) (stroke (width 0) (type default)))

Commit message: Routing R6a-R6m adopted into project board; ERC cleanup, MCU pin swaps, C241 2.2uF, SW100 footprint fix, reviews and helpers
Co-Authored-By: Claude Sonnet 5.5 <noreply@anthropic.com>
Claude-Session: https://claude.ai/code/session_016fe4xPJbEE2SjGafuyNLjb
Parts:
- C241: value 1uF -> 2.2uF; LCSC C29266 -> (none); MPN CL05A105KO5NNNC -> CL05A225KP5NNNC
Changed lines of the file:
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@@
 (wire (pts (xy 271.78 80.01) (xy 264.16 80.01)) (stroke (width 0) (type default)))
 (label "3V3_AUDIO" (at 271.78 80.01 0) (effects (font (size 1 1)) (justify left bottom)))
-(symbol (lib_id "PD_C:PD_C") (at 264.16 83.82 0) (unit 1) (exclude_from_sim no) (in_bom yes) (on_board yes) (dnp no) (property "Reference" "C241" (at 265.43 82.55 0) (effects (font (size 1.27 1.27)) (justify left))) (property "Value" "1uF" (at 265.43 85.09 0) (effects (font (size 1.27 1.27)) (justify left))) (property "Footprint" "DesktopSpeaker:C_0402_1005Metric_Pad0.74x0.62mm_HandSolder" (at 264.16 83.82 0) (hide yes) (effects (font (size 1.27 1.27)))) (property "MPN" "CL05A105KO5NNNC" (at 264.16 83.82 0) (hide yes) (effects (font (size 1.27 1.27)))) (property "Manufacturer" "Samsung Electro-Mechanics" (at 264.16 83.82 0) (hide yes) (effects (font (size 1 1)))) (property "LCSC" "C29266" (at 264.16 83.82 0) (hide yes) (effects (font (size 1 1)))) (pin "1") (pin "2") (instances (project "DesktopSpeaker" (path "/feda53ed-537d-4f88-9436-c6075776255b/07901b33-a7e7-4327-b949-fc2abc1e14b5" (reference "C241") (unit 1)))))
+(symbol (lib_id "PD_C:PD_C") (at 264.16 83.82 0) (unit 1) (exclude_from_sim no) (in_bom yes) (on_board yes) (dnp no) (property "Reference" "C241" (at 265.43 82.55 0) (effects (font (size 1.27 1.27)) (justify left))) (property "Value" "2.2uF" (at 265.43 85.09 0) (effects (font (size 1.27 1.27)) (justify left))) (property "Footprint" "DesktopSpeaker:C_0402_1005Metric_Pad0.74x0.62mm_HandSolder" (at 264.16 83.82 0) (hide yes) (effects (font (size 1.27 1.27)))) (property "MPN" "CL05A225KP5NNNC" (at 264.16 83.82 0) (hide yes) (effects (font (size 1.27 1.27)))) (property "Manufacturer" "Samsung Electro-Mechanics" (at 264.16 83.82 0) (hide yes) (effects (font (size 1 1)))) (property "LCSC" "" (at 264.16 83.82 0) (hide yes) (effects (font (size 1 1)))) (pin "1") (pin "2") (instances (project "DesktopSpeaker" (path "/feda53ed-537d-4f88-9436-c6075776255b/07901b33-a7e7-4327-b949-fc2abc1e14b5" (reference "C241") (unit 1)))))
 (symbol (lib_id "power:GND") (at 264.16 87.63 0) (unit 1) (exclude_from_sim no) (in_bom no) (on_board no) (dnp no) (property "Reference" "#PWR1005" (at 264.16 91.44 0) (effects (font (size 1.27 1.27)) (hide yes))) (property "Value" "GND" (at 264.16 92.71 0) (effects (font (size 1.27 1.27)) (hide yes))) (pin "1") (instances (project "DesktopSpeaker" (path "/feda53ed-537d-4f88-9436-c6075776255b/07901b33-a7e7-4327-b949-fc2abc1e14b5" (reference "#PWR1005") (unit 1)))))
 (symbol (lib_id "power:GND") (at 269.24 146.05 0) (unit 1) (exclude_from_sim no) (in_bom no) (on_board no) (dnp no) (property "Reference" "#PWR1007" (at 269.24 149.86 0) (effects (font (size 1.27 1.27)) (hide yes))) (property "Value" "GND" (at 269.24 151.13 0) (effects (font (size 1.27 1.27)) (hide yes))) (pin "1") (instances (project "DesktopSpeaker" (path "/feda53ed-537d-4f88-9436-c6075776255b/07901b33-a7e7-4327-b949-fc2abc1e14b5" (reference "#PWR1007") (unit 1)))))

Commit message: Y200 24.576 MHz crystal with 15 pF load caps, C275 3D model, schematic/PCB sourcing fields synced to BOM
Co-Authored-By: Claude Sonnet 5.5 <noreply@anthropic.com>
Claude-Session: https://claude.ai/code/session_016fe4xPJbEE2SjGafuyNLjb
Parts:
- C236: LCSC (none) -> C1779
- C241, C243, C244: LCSC (none) -> C7464343
- D200, D201: Manufacturer Nexperia -> DOWO
- R226, R227, R228, R229, R230, R231, R240: LCSC (none) -> C106235
- R232, R233: LCSC (none) -> C93943
- R241: LCSC (none) -> C138033
