File: DesktopSpeaker-kicad/Logic_Audio_Power.kicad_sch (KiCad schematic)
At the start: 9 parts, among them U14 TPS63802DLAR

Commit message: Repackage passives to 0402/0805 hand-solder footprints; update BOM and flags
Co-Authored-By: Claude Sonnet 5.5 <noreply@anthropic.com>
Claude-Session: https://claude.ai/code/session_01N5RHheWSjDFDPbKVD5YVeJ
Parts:
- C140, C141, C142: footprint DesktopSpeaker:PD_C_0805 -> DesktopSpeaker:C_0805_2012Metric_Pad1.18x1.45mm_HandSolder; LCSC (none) -> C907991; Manufacturer (none) -> Murata
- C143: footprint DesktopSpeaker:PD_C_0603 -> DesktopSpeaker:C_0402_1005Metric_Pad0.74x0.62mm_HandSolder; LCSC C1591 -> C77020; LCSC Part C1591 -> C77020; MPN CL10B104KB8NNNC -> GRM155R71H104KE14D; Manufacturer Samsung Electro-Mechanics -> Murata
- R140: footprint DesktopSpeaker:PD_R_0603 -> DesktopSpeaker:R_0402_1005Metric_Pad0.72x0.64mm_HandSolder; LCSC C54531588 -> (none); LCSC Part C54531588 -> (none); MPN 1RC0603F7872 -> RC0402FR-0778K7L; Manufacturer SAE -> Yageo
- R141: footprint DesktopSpeaker:PD_R_0603 -> DesktopSpeaker:R_0402_1005Metric_Pad0.72x0.64mm_HandSolder; LCSC C114639 -> (none); LCSC Part C114639 -> (none); MPN RC0603FR-079K1L -> RC0402FR-079K1L; Manufacturer YAGEO -> Yageo
- R142: footprint DesktopSpeaker:PD_R_0603 -> DesktopSpeaker:R_0402_1005Metric_Pad0.72x0.64mm_HandSolder; LCSC C14675 -> C60491; LCSC Part C14675 -> C60491; MPN RC0603FR-07100KL -> RC0402FR-07100KL; Manufacturer YAGEO -> Yageo

Commit message: Apply low-risk passive cuts (11 parts) and normalise BOM; add layout rules and BOM audit reports
Co-Authored-By: Claude Sonnet 5.5 <noreply@anthropic.com>
Claude-Session: https://claude.ai/code/session_01N5RHheWSjDFDPbKVD5YVeJ
Parts:
- removed C143: 100nF 10V X7R, DesktopSpeaker:C_0402_1005Metric_Pad0.74x0.62mm_HandSolder, symbol PD_C:PD_C
Changed lines of the file:
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@@
 (symbol (lib_id "PD_C:PD_C") (at 208.28 81.28 0) (unit 1) (exclude_from_sim no) (in_bom yes) (on_board yes) (dnp no) (property "Reference" "C141" (at 212.28 80.01 0) (effects (font (size 1.27 1.27)) (justify left))) (property "Value" "22uF 10V X7R" (at 212.28 82.55 0) (effects (font (size 1.27 1.27)) (justify left))) (property "Footprint" "DesktopSpeaker:C_0805_2012Metric_Pad1.18x1.45mm_HandSolder" (at 208.28 81.28 0) (effects (font (size 1.27 1.27)) (hide yes))) (property "LCSC" "C907991" (at 208.28 81.28 0) (hide yes) (effects (font (size 1 1)))) (property "Manufacturer" "Murata" (at 208.28 81.28 0) (hide yes) (effects (font (size 1 1)))) (property "MPN" "GRM21BZ71A226ME15L" (at 208.28 81.28 0) (effects (font (size 1.27 1.27)) (hide yes))) (property "LCSC Part" "C907991" (at 208.28 81.28 0) (effects (font (size 1.27 1.27)) (hide yes))) (pin "1") (pin "2") (instances (project "DesktopSpeaker" (path "/feda53ed-537d-4f88-9436-c6075776255b/31d56ed5-71f9-4c5a-b590-b5d5119f00f9" (reference "C141") (unit 1)))))
 (symbol (lib_id "PD_C:PD_C") (at 231.14 81.28 0) (unit 1) (exclude_from_sim no) (in_bom yes) (on_board yes) (dnp no) (property "Reference" "C142" (at 235.14 80.01 0) (effects (font (size 1.27 1.27)) (justify left))) (property "Value" "22uF 10V X7R" (at 235.14 82.55 0) (effects (font (size 1.27 1.27)) (justify left))) (property "Footprint" "DesktopSpeaker:C_0805_2012Metric_Pad1.18x1.45mm_HandSolder" (at 231.14 81.28 0) (effects (font (size 1.27 1.27)) (hide yes))) (property "LCSC" "C907991" (at 231.14 81.28 0) (hide yes) (effects (font (size 1 1)))) (property "Manufacturer" "Murata" (at 231.14 81.28 0) (hide yes) (effects (font (size 1 1)))) (property "MPN" "GRM21BZ71A226ME15L" (at 231.14 81.28 0) (effects (font (size 1.27 1.27)) (hide yes))) (property "LCSC Part" "C907991" (at 231.14 81.28 0) (effects (font (size 1.27 1.27)) (hide yes))) (pin "1") (pin "2") (instances (project "DesktopSpeaker" (path "/feda53ed-537d-4f88-9436-c6075776255b/31d56ed5-71f9-4c5a-b590-b5d5119f00f9" (reference "C142") (unit 1)))))
-(symbol (lib_id "PD_C:PD_C") (at 118.11 58.42 0) (unit 1) (exclude_from_sim no) (in_bom yes) (on_board yes) (dnp no) (property "Reference" "C143" (at 122.11 57.15 0) (effects (font (size 1.27 1.27)) (justify left))) (property "Value" "100nF 10V X7R" (at 122.11 59.690000000000005 0) (effects (font (size 1.27 1.27)) (justify left))) (property "Footprint" "DesktopSpeaker:C_0402_1005Metric_Pad0.74x0.62mm_HandSolder" (at 118.11 58.42 0) (effects (font (size 1.27 1.27)) (hide yes))) (property "MPN" "GRM155R71H104KE14D" (at 118.11 58.42 0) (effects (font (size 1.27 1.27)) (hide yes))) (property "LCSC Part" "C77020" (at 118.11 58.42 0) (effects (font (size 1.27 1.27)) (hide yes))) (pin "1") (pin "2") (instances (project "DesktopSpeaker" (path "/feda53ed-537d-4f88-9436-c6075776255b/31d56ed5-71f9-4c5a-b590-b5d5119f00f9" (reference "C143") (unit 1)))) (property "Manufacturer" "Murata" (at 118.11 58.42 0) (effects (font (size 1 1)) (hide yes))) (property "LCSC" "C77020" (at 118.11 58.42 0) (effects (font (size 1 1)) (hide yes))) (property "Datasheet" "${KIPRJMOD}/../ai-files/datasheets/Samsung_MLCC_LCSC_C1591_C1711.pdf" (at 118.11 58.42 0) (effects (font (size 1 1)) (hide yes))))
 (symbol (lib_id "PD_R:PD_R") (at 187.96 93.98 0) (unit 1) (exclude_from_sim no) (in_bom yes) (on_board yes) (dnp no) (property "Reference" "R140" (at 191.96 92.71000000000001 0) (effects (font (size 1.27 1.27)) (justify left))) (property "Value" "78.7k 1%" (at 191.96 95.25 0) (effects (font (size 1.27 1.27)) (justify left))) (property "Footprint" "DesktopSpeaker:R_0402_1005Metric_Pad0.72x0.64mm_HandSolder" (at 187.96 93.98 0) (effects (font (size 1.27 1.27)) (hide yes))) (property "MPN" "RC0402FR-0778K7L" (at 187.96 93.98 0) (effects (font (size 1.27 1.27)) (hide yes))) (property "LCSC Part" "" (at 187.96 93.98 0) (effects (font (size 1.27 1.27)) (hide yes))) (pin "1") (pin "2") (instances (project "DesktopSpeaker" (path "/feda53ed-537d-4f88-9436-c6075776255b/31d56ed5-71f9-4c5a-b590-b5d5119f00f9" (reference "R140") (unit 1)))) (property "Manufacturer" "Yageo" (at 187.96 93.98 0) (effects (font (size 1 1)) (hide yes))) (property "LCSC" "" (at 187.96 93.98 0) (effects (font (size 1 1)) (hide yes))) (property "Datasheet" "${KIPRJMOD}/../ai-files/datasheets/SAE_C54531588_1RC0603F7872.pdf" (at 187.96 93.98 0) (effects (font (size 1 1)) (hide yes))))
 (symbol (lib_id "PD_R:PD_R") (at 187.96 118.11 0) (unit 1) (exclude_from_sim no) (in_bom yes) (on_board yes) (dnp no) (property "Reference" "R141" (at 191.96 116.84 0) (effects (font (size 1.27 1.27)) (justify left))) (property "Value" "9.1k 1%" (at 191.96 119.38 0) (effects (font (size 1.27 1.27)) (justify left))) (property "Footprint" "DesktopSpeaker:R_0402_1005Metric_Pad0.72x0.64mm_HandSolder" (at 187.96 118.11 0) (effects (font (size 1.27 1.27)) (hide yes))) (property "MPN" "RC0402FR-079K1L" (at 187.96 118.11 0) (effects (font (size 1.27 1.27)) (hide yes))) (property "LCSC Part" "" (at 187.96 118.11 0) (effects (font (size 1.27 1.27)) (hide yes))) (pin "1") (pin "2") (instances (project "DesktopSpeaker" (path "/feda53ed-537d-4f88-9436-c6075776255b/31d56ed5-71f9-4c5a-b590-b5d5119f00f9" (reference "R141") (unit 1)))) (property "Manufacturer" "Yageo" (at 187.96 118.11 0) (effects (font (size 1 1)) (hide yes))) (property "LCSC" "" (at 187.96 118.11 0) (effects (font (size 1 1)) (hide yes))) (property "Datasheet" "${KIPRJMOD}/../ai-files/datasheets/YAGEO_C114639_RC0603FR-079K1L.pdf" (at 187.96 118.11 0) (effects (font (size 1 1)) (hide yes))))
@@
 (wire (pts (xy 25.4 43.18) (xy 76.2 43.18)) (stroke (width 0) (type default)))
 (wire (pts (xy 76.2 43.18) (xy 101.6 43.18)) (stroke (width 0) (type default)))
-(wire (pts (xy 101.6 43.18) (xy 118.11 43.18)) (stroke (width 0) (type default)))
 (wire (pts (xy 76.2 43.18) (xy 76.2 54.61)) (stroke (width 0) (type default)))
 (junction (at 76.2 43.18) (diameter 0) (color 0 0 0 0))
 (wire (pts (xy 76.2 62.23) (xy 76.2 67.31)) (stroke (width 0) (type default)))
 (symbol (lib_id "power:GND") (at 76.2 67.31 0) (unit 1) (exclude_from_sim no) (in_bom no) (on_board no) (dnp no) (property "Reference" "#PWR140" (at 76.2 71.12 0) (effects (font (size 1.27 1.27)) (hide yes))) (property "Value" "GND" (at 76.2 72.39 0) (effects (font (size 1.27 1.27)))) (pin "1") (instances (project "DesktopSpeaker" (path "/feda53ed-537d-4f88-9436-c6075776255b/31d56ed5-71f9-4c5a-b590-b5d5119f00f9" (reference "#PWR140") (unit 1)))))
-(wire (pts (xy 118.11 43.18) (xy 118.11 54.61)) (stroke (width 0) (type default)))
-(junction (at 118.11 43.18) (diameter 0) (color 0 0 0 0))
-(wire (pts (xy 118.11 62.23) (xy 118.11 67.31)) (stroke (width 0) (type default)))
-(symbol (lib_id "power:GND") (at 118.11 67.31 0) (unit 1) (exclude_from_sim no) (in_bom no) (on_board no) (dnp no) (property "Reference" "#PWR141" (at 118.11 71.12 0) (effects (font (size 1.27 1.27)) (hide yes))) (property "Value" "GND" (at 118.11 72.39 0) (effects (font (size 1.27 1.27)))) (pin "1") (instances (project "DesktopSpeaker" (path "/feda53ed-537d-4f88-9436-c6075776255b/31d56ed5-71f9-4c5a-b590-b5d5119f00f9" (reference "#PWR141") (unit 1)))))
 (wire (pts (xy 101.6 43.18) (xy 101.6 88.9)) (stroke (width 0) (type default)))
-(junction (at 101.6 43.18) (diameter 0) (color 0 0 0 0))
 (wire (pts (xy 25.4 114.3) (xy 69.85 114.3)) (stroke (width 0) (type default)))
 (wire (pts (xy 69.85 114.3) (xy 88.9 114.3)) (stroke (width 0) (type default)))

Commit message: Placement v9: EC11E volume encoder, 25 test points, silkscreen pass (closed sections, border, hole squares, labels), Orwellian logo on back, CAD refit
Co-Authored-By: Claude Sonnet 5.5 <noreply@anthropic.com>
Claude-Session: https://claude.ai/code/session_016fe4xPJbEE2SjGafuyNLjb
Parts:
- added TP7: 5V_LOGIC, DesktopSpeaker:TestPoint_Keystone_5015_Micro_Mini, symbol TestPoint:TestPoint
Connections:
- net 5V_LOGIC: now also TP7.1
Changed lines of the file:
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@@
 (wire (pts (xy 101.6 101.6) (xy 124.46 101.6)) (stroke (width 0) (type default)))
 (wire (pts (xy 139.7 115.57) (xy 142.24 115.57)) (stroke (width 0) (type default)))
-(junction (at 139.7 115.57) (diameter 0) (color 0 0 0 0)))
+(junction (at 139.7 115.57) (diameter 0) (color 0 0 0 0))(symbol (lib_id "TestPoint:TestPoint") (at 254 55.88 0) (unit 1) (exclude_from_sim no) (in_bom no) (on_board yes) (dnp no) (property "Reference" "TP7" (at 256.03 51.31 0) (effects (font (size 1.27 1.27)) (justify left))) (property "Value" "5V_LOGIC" (at 256.03 53.85 0) (effects (font (size 1.27 1.27)) (justify left))) (property "Footprint" "DesktopSpeaker:TestPoint_Keystone_5015_Micro_Mini" (at 254 55.88 0) (hide yes) (effects (font (size 1.27 1.27)))) (property "Datasheet" "" (at 254 55.88 0) (hide yes) (effects (font (size 1.27 1.27)))) (property "Description" "Debug test point (excluded from BOM; hand-fitted loop)" (at 254 55.88 0) (hide yes) (effects (font (size 1 1)))) (pin "1") (instances (project "DesktopSpeaker" (path "/feda53ed-537d-4f88-9436-c6075776255b/31d56ed5-71f9-4c5a-b590-b5d5119f00f9" (reference "TP7") (unit 1)))))
+(wire (pts (xy 254 55.88) (xy 254 58.42)) (stroke (width 0) (type default)))
+(label "5V_LOGIC" (at 254 58.42 0) (effects (font (size 1 1)) (justify left bottom)))
+)

Commit message: Y200 24.576 MHz crystal with 15 pF load caps, C275 3D model, schematic/PCB sourcing fields synced to BOM
Co-Authored-By: Claude Sonnet 5.5 <noreply@anthropic.com>
Claude-Session: https://claude.ai/code/session_016fe4xPJbEE2SjGafuyNLjb
Parts:
- L2: Manufacturer (none) -> Coilcraft
- R140: LCSC (none) -> C163454; LCSC Part (none) -> C163454
- R141: LCSC (none) -> C163450; LCSC Part (none) -> C163450
- U14: Manufacturer (none) -> Texas Instruments
