File: DesktopSpeaker-kicad/Source_Select_ADC.kicad_sch (KiCad schematic)
At the start: 46 parts, among them U22 TPS7A2033PDBVR, U23 TPS22917DBVR, U24 PCM1862DBTR, Y200 24.576MHz

Commit message: Capture Headphone_Aux sheet (TS5A23157 mux, TPA6132A2, jacks) and wire MCU headphone signals
Co-Authored-By: Claude Sonnet 5.5 <noreply@anthropic.com>
Claude-Session: https://claude.ai/code/session_01N5RHheWSjDFDPbKVD5YVeJ
Parts:
- C200, C201, C202, C203, C204, C205: LCSC (none) -> C19110
- C226, C227: value 20pF C0G -> 22pF C0G; LCSC (none) -> C1653; MPN CL10C200JB8NNNC -> CL10C220JB8NNNC
- R200, R201, R202, R203, R204, R205: LCSC (none) -> C105588
- R209, R210: LCSC (none) -> C114662
Other:
- note added: "Crystal CL 15 pF (Lucki L327S240P11L): 2 x 22 pF with about 3 pF stray gives about 14 pF; trim at bring-up. Spare VIN4, MICBIAS and GPIO0/2/3 are no-connect."
- note removed: "Crystal CL 15 pF (Lucki L327S240P11L): 2 x 20 pF with about 3 pF stray gives about 13 pF; trim at bring-up. Spare VIN4, MICBIAS and GPIO0/2/3 are no-connect."

Commit message: Repackage passives to 0402/0805 hand-solder footprints; update BOM and flags
Co-Authored-By: Claude Sonnet 5.5 <noreply@anthropic.com>
Claude-Session: https://claude.ai/code/session_01N5RHheWSjDFDPbKVD5YVeJ
Parts:
- C200, C201, C202, C203, C204, C205: footprint DesktopSpeaker:PD_C_0805 -> DesktopSpeaker:C_0402_1005Metric_Pad0.74x0.62mm_HandSolder; LCSC C19110 -> (none); MPN CL21B225KAFNNNE -> CL05A225KP5NNNC
- C206, C207, C208, C209, C210, C211: footprint DesktopSpeaker:PD_C_0603 -> DesktopSpeaker:C_0402_1005Metric_Pad0.74x0.62mm_HandSolder; MPN GRM1885C1H103JA01D -> GRM1555C1H103JA01D
- C212, C220, C221, C222, C224, C225: footprint DesktopSpeaker:PD_C_0805 -> DesktopSpeaker:C_0402_1005Metric_Pad0.74x0.62mm_HandSolder; LCSC C28323 -> C29266; MPN CL21B105KBFNNNE -> CL05A105KO5NNNC
- C213, C215, C217, C219: footprint DesktopSpeaker:PD_C_0603 -> DesktopSpeaker:C_0402_1005Metric_Pad0.74x0.62mm_HandSolder; LCSC C1591 -> C77020; MPN CL10B104KB8NNNC -> GRM155R71H104KE14D; Manufacturer Samsung Electro-Mechanics -> Murata
- C214, C216, C218, C223: footprint DesktopSpeaker:PD_C_0805 -> DesktopSpeaker:C_0805_2012Metric_Pad1.18x1.45mm_HandSolder
- C226, C227: footprint DesktopSpeaker:PD_C_0603 -> DesktopSpeaker:C_0402_1005Metric_Pad0.74x0.62mm_HandSolder; LCSC C1653 -> (none); MPN CL10C220JB8NNNC -> GRM1555C1H220JA01D; Manufacturer Samsung Electro-Mechanics -> Murata
- FB200: value BLM18AG601SN1D -> BLM15AG601SN1D; footprint DesktopSpeaker:PD_R_0603 -> DesktopSpeaker:R_0402_1005Metric_Pad0.72x0.64mm_HandSolder; LCSC C19330 -> (none); MPN BLM18AG601SN1D -> BLM15AG601SN1D
- R200, R201, R202, R203, R204, R205: footprint DesktopSpeaker:PD_R_0603 -> DesktopSpeaker:R_0402_1005Metric_Pad0.72x0.64mm_HandSolder; LCSC C105588 -> (none); MPN RC0603FR-07100RL -> RC0402FR-07100RL; Manufacturer YAGEO -> Yageo
- R206, R207, R208: footprint DesktopSpeaker:PD_R_0603 -> DesktopSpeaker:R_0402_1005Metric_Pad0.72x0.64mm_HandSolder; MPN RC0603FR-0733RL -> RC0402FR-0733RL; Manufacturer YAGEO -> Yageo
- R209, R210: footprint DesktopSpeaker:PD_R_0603 -> DesktopSpeaker:R_0402_1005Metric_Pad0.72x0.64mm_HandSolder; LCSC C114662 -> (none); MPN RC0603FR-072K2L -> RC0402FR-072K2L; Manufacturer YAGEO -> Yageo
- R211, R212: footprint DesktopSpeaker:PD_R_0603 -> DesktopSpeaker:R_0402_1005Metric_Pad0.72x0.64mm_HandSolder; LCSC C14675 -> C60491; MPN RC0603FR-07100KL -> RC0402FR-07100KL; Manufacturer YAGEO -> Yageo

Commit message: Placement v9: EC11E volume encoder, 25 test points, silkscreen pass (closed sections, border, hole squares, labels), Orwellian logo on back, CAD refit
Co-Authored-By: Claude Sonnet 5.5 <noreply@anthropic.com>
Claude-Session: https://claude.ai/code/session_016fe4xPJbEE2SjGafuyNLjb
Parts:
- added TP12: I2S_BCK, DesktopSpeaker:TestPoint_Keystone_5015_Micro_Mini, symbol TestPoint:TestPoint
- added TP13: I2S_LRCK, DesktopSpeaker:TestPoint_Keystone_5015_Micro_Mini, symbol TestPoint:TestPoint
- added TP14: I2S_SDATA, DesktopSpeaker:TestPoint_Keystone_5015_Micro_Mini, symbol TestPoint:TestPoint
- added TP6: 3V3_AUDIO, DesktopSpeaker:TestPoint_Keystone_5015_Micro_Mini, symbol TestPoint:TestPoint
- added TP8: 5V_CODEC, DesktopSpeaker:TestPoint_Keystone_5015_Micro_Mini, symbol TestPoint:TestPoint
Connections:
- net 3V3_AUDIO: now also TP6.1
- net 5V_CODEC: now also TP8.1
- net I2S_BCK: now also TP12.1
- net I2S_LRCK: now also TP13.1
- net I2S_SDATA: now also TP14.1
Changed lines of the file:
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@@
 (text "Inputs: 2.2 uF - 100 R - 10 nF C0G (datasheet fig. 61 filter; ~5 mA ESD-diode limit). AVDD via FB200. No reset pin: firmware re-initialises after every 3V3_AUDIO enable." (at 129.54 20.32 0) (effects (font (size 1 1)) (justify left bottom)))
 (text "Crystal CL 15 pF (Lucki L327S240P11L): 2 x 22 pF with about 3 pF stray gives about 14 pF; trim at bring-up. Spare VIN4, MICBIAS and GPIO0/2/3 are no-connect." (at 129.54 22.86 0) (effects (font (size 1 1)) (justify left bottom)))
+(symbol (lib_id "TestPoint:TestPoint") (at 284.48 66.04 0) (unit 1) (exclude_from_sim no) (in_bom no) (on_board yes) (dnp no) (property "Reference" "TP6" (at 286.51 61.47 0) (effects (font (size 1.27 1.27)) (justify left))) (property "Value" "3V3_AUDIO" (at 286.51 64.01 0) (effects (font (size 1.27 1.27)) (justify left))) (property "Footprint" "DesktopSpeaker:TestPoint_Keystone_5015_Micro_Mini" (at 284.48 66.04 0) (hide yes) (effects (font (size 1.27 1.27)))) (property "Datasheet" "" (at 284.48 66.04 0) (hide yes) (effects (font (size 1.27 1.27)))) (property "Description" "Debug test point (excluded from BOM; hand-fitted loop)" (at 284.48 66.04 0) (hide yes) (effects (font (size 1 1)))) (pin "1") (instances (project "DesktopSpeaker" (path "/feda53ed-537d-4f88-9436-c6075776255b/d9a0d73a-f008-4736-b4b9-6b3427051836" (reference "TP6") (unit 1)))))
+(wire (pts (xy 284.48 66.04) (xy 284.48 68.58)) (stroke (width 0) (type default)))
+(label "3V3_AUDIO" (at 284.48 68.58 0) (effects (font (size 1 1)) (justify left bottom)))
+(symbol (lib_id "TestPoint:TestPoint") (at 284.48 38.1 0) (unit 1) (exclude_from_sim no) (in_bom no) (on_board yes) (dnp no) (property "Reference" "TP8" (at 286.51 33.53 0) (effects (font (size 1.27 1.27)) (justify left))) (property "Value" "5V_CODEC" (at 286.51 36.07 0) (effects (font (size 1.27 1.27)) (justify left))) (property "Footprint" "DesktopSpeaker:TestPoint_Keystone_5015_Micro_Mini" (at 284.48 38.1 0) (hide yes) (effects (font (size 1.27 1.27)))) (property "Datasheet" "" (at 284.48 38.1 0) (hide yes) (effects (font (size 1.27 1.27)))) (property "Description" "Debug test point (excluded from BOM; hand-fitted loop)" (at 284.48 38.1 0) (hide yes) (effects (font (size 1 1)))) (pin "1") (instances (project "DesktopSpeaker" (path "/feda53ed-537d-4f88-9436-c6075776255b/d9a0d73a-f008-4736-b4b9-6b3427051836" (reference "TP8") (unit 1)))))
+(wire (pts (xy 284.48 38.1) (xy 284.48 40.64)) (stroke (width 0) (type default)))
+(label "5V_CODEC" (at 284.48 40.64 0) (effects (font (size 1 1)) (justify left bottom)))
+(symbol (lib_id "TestPoint:TestPoint") (at 297.18 127 0) (unit 1) (exclude_from_sim no) (in_bom no) (on_board yes) (dnp no) (property "Reference" "TP12" (at 299.21 122.43 0) (effects (font (size 1.27 1.27)) (justify left))) (property "Value" "I2S_BCK" (at 299.21 124.97 0) (effects (font (size 1.27 1.27)) (justify left))) (property "Footprint" "DesktopSpeaker:TestPoint_Keystone_5015_Micro_Mini" (at 297.18 127 0) (hide yes) (effects (font (size 1.27 1.27)))) (property "Datasheet" "" (at 297.18 127 0) (hide yes) (effects (font (size 1.27 1.27)))) (property "Description" "Debug test point (excluded from BOM; hand-fitted loop)" (at 297.18 127 0) (hide yes) (effects (font (size 1 1)))) (pin "1") (instances (project "DesktopSpeaker" (path "/feda53ed-537d-4f88-9436-c6075776255b/d9a0d73a-f008-4736-b4b9-6b3427051836" (reference "TP12") (unit 1)))))
+(wire (pts (xy 297.18 127) (xy 297.18 129.54)) (stroke (width 0) (type default)))
+(label "I2S_BCK" (at 297.18 129.54 0) (effects (font (size 1 1)) (justify left bottom)))
+(symbol (lib_id "TestPoint:TestPoint") (at 284.48 144.78 0) (unit 1) (exclude_from_sim no) (in_bom no) (on_board yes) (dnp no) (property "Reference" "TP13" (at 286.51 140.21 0) (effects (font (size 1.27 1.27)) (justify left))) (property "Value" "I2S_LRCK" (at 286.51 142.75 0) (effects (font (size 1.27 1.27)) (justify left))) (property "Footprint" "DesktopSpeaker:TestPoint_Keystone_5015_Micro_Mini" (at 284.48 144.78 0) (hide yes) (effects (font (size 1.27 1.27)))) (property "Datasheet" "" (at 284.48 144.78 0) (hide yes) (effects (font (size 1.27 1.27)))) (property "Description" "Debug test point (excluded from BOM; hand-fitted loop)" (at 284.48 144.78 0) (hide yes) (effects (font (size 1 1)))) (pin "1") (instances (project "DesktopSpeaker" (path "/feda53ed-537d-4f88-9436-c6075776255b/d9a0d73a-f008-4736-b4b9-6b3427051836" (reference "TP13") (unit 1)))))
+(wire (pts (xy 284.48 144.78) (xy 284.48 147.32)) (stroke (width 0) (type default)))
+(label "I2S_LRCK" (at 284.48 147.32 0) (effects (font (size 1 1)) (justify left bottom)))
+(symbol (lib_id "TestPoint:TestPoint") (at 284.48 111.76 0) (unit 1) (exclude_from_sim no) (in_bom no) (on_board yes) (dnp no) (property "Reference" "TP14" (at 286.51 107.19 0) (effects (font (size 1.27 1.27)) (justify left))) (property "Value" "I2S_SDATA" (at 286.51 109.73 0) (effects (font (size 1.27 1.27)) (justify left))) (property "Footprint" "DesktopSpeaker:TestPoint_Keystone_5015_Micro_Mini" (at 284.48 111.76 0) (hide yes) (effects (font (size 1.27 1.27)))) (property "Datasheet" "" (at 284.48 111.76 0) (hide yes) (effects (font (size 1.27 1.27)))) (property "Description" "Debug test point (excluded from BOM; hand-fitted loop)" (at 284.48 111.76 0) (hide yes) (effects (font (size 1 1)))) (pin "1") (instances (project "DesktopSpeaker" (path "/feda53ed-537d-4f88-9436-c6075776255b/d9a0d73a-f008-4736-b4b9-6b3427051836" (reference "TP14") (unit 1)))))
+(wire (pts (xy 284.48 111.76) (xy 284.48 114.3)) (stroke (width 0) (type default)))
+(label "I2S_SDATA" (at 284.48 114.3 0) (effects (font (size 1 1)) (justify left bottom)))
 )

Commit message: Routing R6a-R6m adopted into project board; ERC cleanup, MCU pin swaps, C241 2.2uF, SW100 footprint fix, reviews and helpers
Co-Authored-By: Claude Sonnet 5.5 <noreply@anthropic.com>
Claude-Session: https://claude.ai/code/session_016fe4xPJbEE2SjGafuyNLjb
Parts:
- TP13: value I2S_LRCK -> I2S_SDATA
- TP14: value I2S_SDATA -> I2S_LRCK
Connections:
- net I2S_LRCK: now also TP14.1; no longer TP13.1
- net I2S_SDATA: now also TP13.1; no longer TP14.1
Changed lines of the file:
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@@
 (wire (pts (xy 297.18 127) (xy 297.18 129.54)) (stroke (width 0) (type default)))
 (label "I2S_BCK" (at 297.18 129.54 0) (effects (font (size 1 1)) (justify left bottom)))
-(symbol (lib_id "TestPoint:TestPoint") (at 284.48 144.78 0) (unit 1) (exclude_from_sim no) (in_bom no) (on_board yes) (dnp no) (property "Reference" "TP13" (at 286.51 140.21 0) (effects (font (size 1.27 1.27)) (justify left))) (property "Value" "I2S_LRCK" (at 286.51 142.75 0) (effects (font (size 1.27 1.27)) (justify left))) (property "Footprint" "DesktopSpeaker:TestPoint_Keystone_5015_Micro_Mini" (at 284.48 144.78 0) (hide yes) (effects (font (size 1.27 1.27)))) (property "Datasheet" "" (at 284.48 144.78 0) (hide yes) (effects (font (size 1.27 1.27)))) (property "Description" "Debug test point (excluded from BOM; hand-fitted loop)" (at 284.48 144.78 0) (hide yes) (effects (font (size 1 1)))) (pin "1") (instances (project "DesktopSpeaker" (path "/feda53ed-537d-4f88-9436-c6075776255b/d9a0d73a-f008-4736-b4b9-6b3427051836" (reference "TP13") (unit 1)))))
+(symbol (lib_id "TestPoint:TestPoint") (at 284.48 144.78 0) (unit 1) (exclude_from_sim no) (in_bom no) (on_board yes) (dnp no) (property "Reference" "TP13" (at 286.51 140.21 0) (effects (font (size 1.27 1.27)) (justify left))) (property "Value" "I2S_SDATA" (at 286.51 142.75 0) (effects (font (size 1.27 1.27)) (justify left))) (property "Footprint" "DesktopSpeaker:TestPoint_Keystone_5015_Micro_Mini" (at 284.48 144.78 0) (hide yes) (effects (font (size 1.27 1.27)))) (property "Datasheet" "" (at 284.48 144.78 0) (hide yes) (effects (font (size 1.27 1.27)))) (property "Description" "Debug test point (excluded from BOM; hand-fitted loop)" (at 284.48 144.78 0) (hide yes) (effects (font (size 1 1)))) (pin "1") (instances (project "DesktopSpeaker" (path "/feda53ed-537d-4f88-9436-c6075776255b/d9a0d73a-f008-4736-b4b9-6b3427051836" (reference "TP13") (unit 1)))))
 (wire (pts (xy 284.48 144.78) (xy 284.48 147.32)) (stroke (width 0) (type default)))
-(label "I2S_LRCK" (at 284.48 147.32 0) (effects (font (size 1 1)) (justify left bottom)))
-(symbol (lib_id "TestPoint:TestPoint") (at 284.48 111.76 0) (unit 1) (exclude_from_sim no) (in_bom no) (on_board yes) (dnp no) (property "Reference" "TP14" (at 286.51 107.19 0) (effects (font (size 1.27 1.27)) (justify left))) (property "Value" "I2S_SDATA" (at 286.51 109.73 0) (effects (font (size 1.27 1.27)) (justify left))) (property "Footprint" "DesktopSpeaker:TestPoint_Keystone_5015_Micro_Mini" (at 284.48 111.76 0) (hide yes) (effects (font (size 1.27 1.27)))) (property "Datasheet" "" (at 284.48 111.76 0) (hide yes) (effects (font (size 1.27 1.27)))) (property "Description" "Debug test point (excluded from BOM; hand-fitted loop)" (at 284.48 111.76 0) (hide yes) (effects (font (size 1 1)))) (pin "1") (instances (project "DesktopSpeaker" (path "/feda53ed-537d-4f88-9436-c6075776255b/d9a0d73a-f008-4736-b4b9-6b3427051836" (reference "TP14") (unit 1)))))
+(label "I2S_SDATA" (at 284.48 147.32 0) (effects (font (size 1 1)) (justify left bottom)))
+(symbol (lib_id "TestPoint:TestPoint") (at 284.48 111.76 0) (unit 1) (exclude_from_sim no) (in_bom no) (on_board yes) (dnp no) (property "Reference" "TP14" (at 286.51 107.19 0) (effects (font (size 1.27 1.27)) (justify left))) (property "Value" "I2S_LRCK" (at 286.51 109.73 0) (effects (font (size 1.27 1.27)) (justify left))) (property "Footprint" "DesktopSpeaker:TestPoint_Keystone_5015_Micro_Mini" (at 284.48 111.76 0) (hide yes) (effects (font (size 1.27 1.27)))) (property "Datasheet" "" (at 284.48 111.76 0) (hide yes) (effects (font (size 1.27 1.27)))) (property "Description" "Debug test point (excluded from BOM; hand-fitted loop)" (at 284.48 111.76 0) (hide yes) (effects (font (size 1 1)))) (pin "1") (instances (project "DesktopSpeaker" (path "/feda53ed-537d-4f88-9436-c6075776255b/d9a0d73a-f008-4736-b4b9-6b3427051836" (reference "TP14") (unit 1)))))
 (wire (pts (xy 284.48 111.76) (xy 284.48 114.3)) (stroke (width 0) (type default)))
-(label "I2S_SDATA" (at 284.48 114.3 0) (effects (font (size 1 1)) (justify left bottom)))
+(label "I2S_LRCK" (at 284.48 114.3 0) (effects (font (size 1 1)) (justify left bottom)))
 )

Commit message: Y200 24.576 MHz crystal with 15 pF load caps, C275 3D model, schematic/PCB sourcing fields synced to BOM
Co-Authored-By: Claude Sonnet 5.5 <noreply@anthropic.com>
Claude-Session: https://claude.ai/code/session_016fe4xPJbEE2SjGafuyNLjb
Parts:
- C200, C201, C202, C203, C204, C205: LCSC (none) -> C7464343
- C206, C207, C208, C209, C210, C211: LCSC (none) -> C22400107; MPN GRM1555C1H103JA01D -> GRM1555C1H103JE01D
- C226, C227: value 22pF C0G -> 15pF C0G; LCSC (none) -> C76950; MPN GRM1555C1H220JA01D -> GRM1555C1H150JA01D
- FB200: LCSC (none) -> C76884
- R200, R201, R202, R203, R204, R205: LCSC (none) -> C106232
- R206, R207, R208: LCSC (none) -> C138002
- R209, R210: LCSC (none) -> C114762
- Y200: LCSC C5261154 -> C70568; MPN L327S240P11L -> X322524576MOB4SI; Manufacturer Lucki -> YXC
