File: ai-files/pcb/DesktopSpeaker-p0-routed.kicad_pcb (KiCad board)
At the start: 4 copper layers, 136.9 x 127.8 mm, 351 parts, among them J1 USB_C_Receptacle_USB2.0_16P, J10 B2P-VH, J11 B2P-VH, J2 HEAD_OUT, J3 AUX_IN, J4 I2C service, J5 1S_PACK_3PIN, J6 SWD, J7 SWD_TC2030, J8 BM83_PROG, J9 B2P-VH, Q100 2N7002, Q101 2N7002, Q102 2N7002, Q103 CSD17579Q3A, Q104 2N7002, SW100 WAKE_QON, SW101 BAT_DISCONNECT, SW102 EC11E, U1 BM83SM1-00TA, U10 TPA6132A2RTER, U11 TPS25730DREFR, U12 TPS7A0230PDBVR, U13 TS5A3167DBVR, U14 TPS63802DLAR, U15 TPS63802DLAR, U16 TS5A3167DBVR, U17 TS5A3167DBVR, U19 TPS7B8450QWDRBRQ1, U2 PCM2902CDBR, U20 TPS2116DRLR, U21 TPS3839G33DBZR, U22 TPS7A2033PDBVR, U23 TPS22917DBVR, U24 PCM1862DBTR, U25 TPS61088RHLR, U3 STM32G071RBT6, U4 BQ25792RQMR, U5 MAX17048G+T10, U6 TAS5825MRHBR, U7 TAS5825MRHBR, U8 TS5A23157DGSR, U9 TS5A23157DGSR, Y170 12MHz, Y200 24.576MHz

Commit message: Routing phase 0: GND planes, In2 rail islands, F.Cu pours, 203 GND vias, rail vias; Freerouting trial (draft, not adopted); routing P0 scripts and report
Co-Authored-By: Claude Sonnet 5.5 <noreply@anthropic.com>
Claude-Session: https://claude.ai/code/session_016fe4xPJbEE2SjGafuyNLjb
Routing:
- net GND: track 159.0 -> 502.5 mm, vias 203 -> 215
- net /5V_LOGIC: track 3.50 -> 109.3 mm, vias 4 -> 7
- net /5V_CODEC: track 3.19 -> 50.8 mm, vias 3 -> 5
- net /3V_AO: track 3.90 -> 45.0 mm, vias 4 -> 5
- net /USB_PD/LDO_3V3: track 0.00 -> 37.2 mm, vias 0 -> 2
- net Net-(U2-VCCCI): track 0.00 -> 9.90 mm, vias 0 -> 2
- net Net-(U24-AVDD): track 0.00 -> 9.11 mm, vias 0 -> 2
- net /Battery_Charger/REGN: track 0.00 -> 8.82 mm
- net Net-(Q104-G): track 0.00 -> 8.29 mm
- net Net-(U2-VCCP2I): track 0.00 -> 7.83 mm, vias 0 -> 2
- net Net-(U2-VBUS): track 0.00 -> 6.50 mm
- net Net-(U14-FB): track 0.00 -> 6.33 mm
- net /CTRL_SDA: track 0.00 -> 5.96 mm
- net Net-(U2-VCCP1I): track 0.00 -> 5.20 mm, vias 0 -> 2
- net Net-(U25-ILIM): track 0.00 -> 4.22 mm
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